File: Electronica/PCB/Clase de Club robotica/Clase de Club robotica.kicad_pcb (KiCad board)
At the start: 2 copper layers, 21 parts, among them J1 Ultrasonico 1, J3 Ultrasonico 2, J4 Ultrasonico 3, J5 Ultrasonico 4, SW1 SW_SPST, SW2 SW_Push, U1 CNY70, U2 CNY70

Commit message: No se
Parts:
- removed R2, R5: 10K, Resistor_THT:R_Axial_DIN0207_L6.3mm_D2.5mm_P10.16mm_Horizontal
- removed R3, R4: 200, Resistor_THT:R_Axial_DIN0207_L6.3mm_D2.5mm_P10.16mm_Horizontal
- moved U2 164.4 mm to (65.2, 97.9), turned to 180 degrees
- moved D2 156.8 mm to (17.0, 66.5), turned to 180 degrees
- moved A2 148.6 mm to (120.8, 164.8), turned to 180 degrees
- moved Conector_Apb1 148.2 mm to (29.6, 82.5), turned to -90 degrees
- moved R1 110.0 mm to (27.1, 74.0), turned to 180 degrees
- moved SensoresPISO2 108.0 mm to (102.6, 76.5), turned to -90 degrees
- moved SW1 101.6 mm to (17.0, 54.2)
- moved D1 83.7 mm to (32.1, 54.0), turned to 180 degrees
- moved U1 66.7 mm to (121.8, 76.0), turned to -90 degrees
- moved U2 65.1 mm to (128.5, 76.1), turned to 180 degrees
- moved SensoresPISO1 55.0 mm to (151.0, 75.9)
- moved SW2 51.8 mm to (138.5, 90.0)
- moved J4 9.69 mm to (128.0, 106.0)
- moved J3 8.80 mm to (123.3, 106.0)
- moved J1 5.55 mm to (123.6, 110.0)
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Connections:
- A1 pad 10: TRIG 1 -> ECHO 1
- A1 pad 15: ECHO 4 -> unconnected-(A1-D12-Pad15)
- A1 pad 16: TRIG 4 -> unconnected-(A1-D13-Pad16)
- A1 pad 21: unconnected-(A1-A2-Pad21) -> BOTON 
- A1 pad 9: ECHO 1 -> TRIG 1
Routing:
- net +5V: track 0.00 -> 374.0 mm
- net GND: track 90.7 -> 182.6 mm
- net PWM B MONSTER SHIELD: track 0.00 -> 83.3 mm
- net SENSOR DE PISO 2: track 0.00 -> 50.5 mm
- net AIN2 MONSTER SHIELD: track 30.5 -> 0.00 mm
- net AIN1 MONSTER SHIELD: track 29.9 -> 0.00 mm
- net BOTON : track 0.00 -> 25.0 mm
- net Earth: track 0.00 -> 22.7 mm
- net TRIG 4: track 0.00 -> 20.1 mm
- net PWM A MONSTER SHIELD: track 0.00 -> 19.2 mm
- net BIN 1 MONSTER SHIELD: track 0.00 -> 19.2 mm
- net VIN: track 0.00 -> 18.8 mm
- net BIN 2 MONSTER SHIELD: track 0.00 -> 16.9 mm
- net TRIG 1: track 9.70 -> 26.2 mm
- net ECHO 4: track 0.00 -> 14.6 mm
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
Commit message: Quedan 4 puentes
Parts:
- removed D1: SB120, Diode_THT:D_DO-41_SOD81_P10.16mm_Horizontal
- removed J5: Ultrasonico 4, Connector_PinHeader_2.54mm:PinHeader_1x04_P2.54mm_Vertical
- removed U1: CNY70, Connector_PinHeader_2.54mm:PinHeader_1x04_P2.54mm_Vertical
- removed the U2 at (128.5, 76.1)
- added SensoresPISO3: Conn_01x04, Connector_PinSocket_2.54mm:PinSocket_1x04_P2.54mm_Vertical, F.Cu at (104.5, 76.5)
- moved SensoresPISO1 43.7 mm to (107.5, 71.5), turned to 180 degrees
- moved SensoresPISO2 6.38 mm to (109.0, 76.5), turned to 90 degrees
Connections:
- A1 pad 1: AIN2 MONSTER SHIELD -> unconnected-(A1-D1/TX-Pad1)
- A1 pad 15: unconnected-(A1-D12-Pad15) -> AIN1 MONSTER SHIELD
- A1 pad 16: unconnected-(A1-D13-Pad16) -> AIN2 MONSTER SHIELD
- A1 pad 2: AIN1 MONSTER SHIELD -> unconnected-(A1-D0/RX-Pad2)
- A1 pad 21: BOTON  -> unconnected-(A1-A2-Pad21)
- A1 pad 22: unconnected-(A1-A3-Pad22) -> BOTON 
- A1 pad 25: unconnected-(A1-A6-Pad25) -> PWM B MONSTER SHIELD
- A1 pad 26: unconnected-(A1-A7-Pad26) -> SENSOR DE PISO 3
- A1 pad 8: PWM B MONSTER SHIELD -> unconnected-(A1-D5-Pad8)
Routing:
- net GND: track 182.6 -> 365.6 mm
- net +5V: track 374.0 -> 279.5 mm
- net AIN2 MONSTER SHIELD: track 0.00 -> 84.0 mm
- net AIN1 MONSTER SHIELD: track 0.00 -> 51.7 mm
- net SENSOR DE PISO 2: track 50.5 -> 9.18 mm
- net SENSOR DE PISO 1: track 0.00 -> 34.4 mm
- net TRIG 4: track 20.1 -> 0.00 mm
- net unconnected-(A1-D5-Pad8): track 0.00 -> 14.7 mm
- net ECHO 4: track 14.6 -> 0.00 mm
- net SENSOR DE PISO 3: track 0.00 -> 11.0 mm
- net unconnected-(A1-D13-Pad16): track 8.49 -> 0.00 mm
- net PWM B MONSTER SHIELD: track 83.3 -> 76.0 mm
- net BOTON : track 25.0 -> 27.6 mm

Commit message: 4 puentes
Connections:
- A1 pad 15: AIN1 MONSTER SHIELD -> unconnected-(A1-D12-Pad15)
- A1 pad 24: unconnected-(A1-A5-Pad24) -> PWM B MONSTER SHIELD
- A1 pad 25: PWM B MONSTER SHIELD -> AIN1 MONSTER SHIELD
Routing:
- net GND: track 365.6 -> 440.3 mm
- net AIN1 MONSTER SHIELD: track 51.7 -> 94.8 mm
- net +5V: track 279.5 -> 312.1 mm
- net unconnected-(A1-D5-Pad8): track 14.7 -> 0.00 mm
- net PWM B MONSTER SHIELD: track 76.0 -> 86.3 mm
