File: Electronica/PCB/Clase de Club robotica/Clase de Club robotica.kicad_pcb (KiCad board)
At the start: 2 copper layers, 5 parts, among them J1 Ultrasonico, SW1 SW_SPST

Commit message: Inicio de diseño del pcb
Parts:
- added Conector_Apb1: Conector Apb, Connector_PinHeader_2.54mm:PinHeader_1x03_P2.54mm_Vertical, F.Cu at (173.5, 46.9)
- added D2: LED, Connector_PinHeader_2.54mm:PinHeader_1x02_P2.54mm_Vertical, F.Cu at (173.5, 56.6)
- added J3: Ultrasonico 2, Connector_PinHeader_2.54mm:PinHeader_1x04_P2.54mm_Vertical, F.Cu at (131.1, 110.0)
- added J4: Ultrasonico 3, Connector_PinHeader_2.54mm:PinHeader_1x04_P2.54mm_Vertical, F.Cu at (136.8, 109.8)
- added J5: Ultrasonico 4, Connector_PinHeader_2.54mm:PinHeader_1x04_P2.54mm_Vertical, F.Cu at (144.8, 95.8)
- added R1: R_US, Resistor_THT:R_Axial_DIN0207_L6.3mm_D2.5mm_P10.16mm_Horizontal, F.Cu at (136.6, 83.5)
- added R2: 10K, Resistor_THT:R_Axial_DIN0207_L6.3mm_D2.5mm_P10.16mm_Horizontal, F.Cu at (159.4, 50.6)
- added R3: 200, Resistor_THT:R_Axial_DIN0207_L6.3mm_D2.5mm_P10.16mm_Horizontal, F.Cu at (159.4, 54.7)
- added R4: 200, Resistor_THT:R_Axial_DIN0207_L6.3mm_D2.5mm_P10.16mm_Horizontal, F.Cu at (159.4, 58.8)
- added R5: 10K, Resistor_THT:R_Axial_DIN0207_L6.3mm_D2.5mm_P10.16mm_Horizontal, F.Cu at (133.5, 78.9)
- added SW2: SW_Push, Connector_PinHeader_2.54mm:PinHeader_1x02_P2.54mm_Vertical, F.Cu at (178.1, 56.6)
- added U1: CNY70, Connector_PinHeader_2.54mm:PinHeader_1x04_P2.54mm_Vertical, F.Cu at (174.1, 34.6)
- added U2: CNY70, Connector_PinHeader_2.54mm:PinHeader_1x04_P2.54mm_Vertical, F.Cu at (178.8, 34.6)
- A2: value Arduino_UNO_R3 -> MONSTER SHIELD
- J1: value Ultrasonico -> Ultrasonico 1
- SW1: footprint Button_Switch_THT:SW_Slide_SPDT_Straight_CK_OS102011MS2Q -> Connector_PinHeader_2.54mm:PinHeader_1x02_P2.54mm_Vertical
- moved J1 83.2 mm to (118.0, 110.0), turned to -90 degrees
- moved A1 77.2 mm to (92.6, 100.3), turned to 90 degrees
Connections:
- A1 pad 1: unconnected-(A1-D1/TX-Pad1) -> AIN2 MONSTER SHIELD
- A1 pad 10: unconnected-(A1-D7-Pad10) -> TRIG 1
- A1 pad 11: unconnected-(A1-D8-Pad11) -> ECHO 2
- A1 pad 12: unconnected-(A1-D9-Pad12) -> TRIG 2
- A1 pad 13: unconnected-(A1-D10-Pad13) -> ECHO 3
- A1 pad 14: unconnected-(A1-D11-Pad14) -> TRIG 3
- A1 pad 15: unconnected-(A1-D12-Pad15) -> ECHO 4
- A1 pad 16: unconnected-(A1-D13-Pad16) -> TRIG 4
- A1 pad 19: unconnected-(A1-A0-Pad19) -> SENSOR DE PISO 1
- A1 pad 2: unconnected-(A1-D0/RX-Pad2) -> AIN1 MONSTER SHIELD
- A1 pad 20: unconnected-(A1-A1-Pad20) -> SENSOR DE PISO 2
- A1 pad 27: unconnected-(A1-+5V-Pad27) -> +5V
- A1 pad 29: unconnected-(A1-GND-Pad29) -> GND
- A1 pad 4: unconnected-(A1-GND-Pad4) -> GND
- A1 pad 5: unconnected-(A1-D2-Pad5) -> BIN 1 MONSTER SHIELD
- A1 pad 6: unconnected-(A1-D3-Pad6) -> PWM A MONSTER SHIELD
- A1 pad 7: unconnected-(A1-D4-Pad7) -> BIN 2 MONSTER SHIELD
- A1 pad 8: unconnected-(A1-D5-Pad8) -> PWM B MONSTER SHIELD
- A1 pad 9: unconnected-(A1-D6-Pad9) -> ECHO 1
- A2 pad 19: unconnected-(A2-D4-Pad19) -> BIN 1 MONSTER SHIELD
- A2 pad 20: unconnected-(A2-D5-Pad20) -> PWM A MONSTER SHIELD
- A2 pad 21: unconnected-(A2-D6-Pad21) -> PWM B MONSTER SHIELD
- A2 pad 22: unconnected-(A2-D7-Pad22) -> AIN1 MONSTER SHIELD
- A2 pad 23: unconnected-(A2-D8-Pad23) -> AIN2 MONSTER SHIELD
- A2 pad 24: unconnected-(A2-D9-Pad24) -> BIN 2 MONSTER SHIELD
- A2 pad 29: unconnected-(A2-GND-Pad29) -> GND
- A2 pad 5: unconnected-(A2-+5V-Pad5) -> +5V
- A2 pad 6: unconnected-(A2-GND-Pad6) -> GND
- A2 pad 7: unconnected-(A2-GND-Pad7) -> GND
- D1 pad 2: unconnected-(D1-A-Pad2) -> Net-(D1-A)
- J1 pad 1: (no net) -> +5V
- J1 pad 2: unconnected-(J1-Pin_2-Pad2) -> TRIG 1
- J1 pad 3: unconnected-(J1-Pin_3-Pad3) -> ECHO 1
- J1 pad 4: unconnected-(J1-Pin_4-Pad4) -> GND
- SW1 pad 1: unconnected-(SW1-A-Pad1) -> Net-(D1-A)
- SW1 pad 2: unconnected-(SW1-B-Pad2) -> Net-(Conector_Apb1-Pin_1)
Routing:
- net GND: track 0.00 -> 90.7 mm
- net AIN2 MONSTER SHIELD: track 0.00 -> 30.5 mm
- net AIN1 MONSTER SHIELD: track 0.00 -> 29.9 mm
- net TRIG 3: track 0.00 -> 21.3 mm
- net ECHO 3: track 0.00 -> 20.9 mm
- net TRIG 2: track 0.00 -> 13.0 mm
- net ECHO 2: track 0.00 -> 13.0 mm
- net TRIG 1: track 0.00 -> 9.70 mm
- net ECHO 1: track 0.00 -> 9.70 mm

Commit message: Huella step Down
Parts:
- added SensoresPISO1: Conn_01x04, Connector_PinSocket_2.54mm:PinSocket_1x04_P2.54mm_Vertical, F.Cu at (206.0, 76.1)
- added SensoresPISO2: Conn_01x04, Connector_PinSocket_2.54mm:PinSocket_1x04_P2.54mm_Vertical, F.Cu at (210.6, 76.1)
- added U2: ~, Step Down:Step Down, F.Cu at (229.3, 87.6)
Connections:
- A1 pad 30: unconnected-(A1-VIN-Pad30) -> VIN
- A2 pad 10: unconnected-(A2-A1-Pad10) -> +5V
- A2 pad 9: unconnected-(A2-A0-Pad9) -> +5V
- D2 pad 2: Net-(Conector_Apb1-Pin_1) -> Net-(D2-A)
- SW1 pad 2: Net-(Conector_Apb1-Pin_1) -> Net-(D2-A)

Commit message: Placa hoy le pregunto a prieto del diseño
Parts:
- removed Conector_Apb1: Conector Apb, Connector_PinHeader_2.54mm:PinHeader_1x03_P2.54mm_Vertical
- removed J5: Ultrasonico 4, Connector_PinHeader_2.54mm:PinHeader_1x04_P2.54mm_Vertical
- removed R2, R5: 10K, Resistor_THT:R_Axial_DIN0207_L6.3mm_D2.5mm_P10.16mm_Horizontal
- removed R3, R4: 200, Resistor_THT:R_Axial_DIN0207_L6.3mm_D2.5mm_P10.16mm_Horizontal
- removed the U2 at (178.8, 34.6)
- added J2: Screw_Terminal_01x02, TerminalBlock:TerminalBlock_bornier-2_P5.08mm, F.Cu at (129.9, 146.0)
- added J6: Screw_Terminal_01x02, Connector_PinSocket_2.54mm:PinSocket_1x02_P2.54mm_Vertical, F.Cu at (139.1, 54.6)
- added SensoresPISO3: Conn_01x04, Connector_PinSocket_2.54mm:PinSocket_1x04_P2.54mm_Vertical, F.Cu at (174.8, 57.2)
- D1: value SB120 -> D; footprint Diode_THT:D_DO-41_SOD81_P10.16mm_Horizontal -> Diode_THT:D_5W_P10.16mm_Horizontal
- U1: value CNY70 -> ~; footprint Connector_PinHeader_2.54mm:PinHeader_1x04_P2.54mm_Vertical -> misc_footprints:MT3608_module
- moved A2 170.4 mm to (191.1, 145.5), turned to 180 degrees
- moved U1 96.8 mm to (127.5, 119.5), turned to 90 degrees
- moved U2 93.6 mm to (135.7, 87.4), turned to 180 degrees
- moved J1 77.3 mm to (193.4, 92.6)
- moved A1 72.9 mm to (162.9, 81.1)
- moved J3 67.0 mm to (193.6, 85.6)
- moved J4 64.8 mm to (198.2, 89.0)
- moved D2 41.6 mm to (131.9, 54.6), turned to -90 degrees
- moved SensoresPISO2 36.6 mm to (179.2, 57.2), turned to 90 degrees
- moved SW2 33.8 mm to (208.8, 70.7)
- moved R1 26.1 mm to (142.2, 58.0), turned to 180 degrees
- moved SW1 22.8 mm to (121.1, 54.4), turned to 90 degrees
- moved SensoresPISO1 20.2 mm to (198.8, 57.2), turned to -90 degrees
- moved D1 7.13 mm to (115.7, 64.1), turned to 90 degrees
Connections:
- A1 pad 1: AIN2 MONSTER SHIELD -> unconnected-(A1-D1/TX-Pad1)
- A1 pad 15: ECHO 4 -> unconnected-(A1-D12-Pad15)
- A1 pad 16: TRIG 4 -> AIN2 MONSTER SHIELD
- A1 pad 2: AIN1 MONSTER SHIELD -> unconnected-(A1-D0/RX-Pad2)
- A1 pad 22: unconnected-(A1-A3-Pad22) -> BOTON 
- A1 pad 24: unconnected-(A1-A5-Pad24) -> PWM B MONSTER SHIELD
- A1 pad 25: unconnected-(A1-A6-Pad25) -> AIN1 MONSTER SHIELD
- A1 pad 26: unconnected-(A1-A7-Pad26) -> SENSOR DE PISO 3
- A1 pad 8: PWM B MONSTER SHIELD -> unconnected-(A1-D5-Pad8)
- D1 pad 1: unconnected-(D1-K-Pad1) -> STEP DOWN
Routing:
- net +5V: track 0.00 -> 347.9 mm
- net GND: track 90.7 -> 349.6 mm
- net Earth: track 0.00 -> 92.4 mm
- net PWM B MONSTER SHIELD: track 0.00 -> 90.5 mm
- net AIN1 MONSTER SHIELD: track 29.9 -> 105.8 mm
- net STEP DOWN: track 0.00 -> 64.8 mm
- net AIN2 MONSTER SHIELD: track 30.5 -> 91.7 mm
- net VIN: track 0.00 -> 39.4 mm
- net BOTON : track 0.00 -> 30.5 mm
- net ECHO 3: track 20.9 -> 48.4 mm
- net PWM A MONSTER SHIELD: track 0.00 -> 23.5 mm
- net BIN 1 MONSTER SHIELD: track 0.00 -> 23.5 mm
- net Net-(D2-A): track 0.00 -> 20.4 mm
- net BIN 2 MONSTER SHIELD: track 0.00 -> 16.9 mm
- net SENSOR DE PISO 3: track 0.00 -> 15.1 mm
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