File: Electronica/PCB/Clase de Club robotica/Clase de Club robotica.kicad_sch (KiCad schematic)
At the start: 18 parts, among them J1 Ultrasonico 1, J3 Ultrasonico 2, J4 Ultrasonico 3, J5 Ultrasonico 4, SW1 SW_SPST, SW2 SW_Push, U1 CNY70, U2 CNY70

Commit message: Inicio de diseño del pcb
Connections:
- net +5V: now also A2.5 (+5V), J4.4 (Pin_4); no longer A2.8 (VIN), J4.1 (Pin_1)
- net ECHO 3: now also J4.2 (Pin_2); no longer J4.3 (Pin_3)
- net GND: now also J4.1 (Pin_1); no longer J4.4 (Pin_4)
- net TRIG 3: now also J4.3 (Pin_3); no longer J4.2 (Pin_2)

Commit message: Esquematico correjido por prieto solo falta el step up y step down
Parts:
- removed Conector_Apb1: Conector Apb, Connector_PinHeader_2.54mm:PinHeader_1x03_P2.54mm_Vertical, symbol Connector_Generic:Conn_01x03
- removed D1: SB120, Diode_THT:D_DO-41_SOD81_P10.16mm_Horizontal, symbol Diode:SB120
- removed R2, R5: 10K, Resistor_THT:R_Axial_DIN0207_L6.3mm_D2.5mm_P10.16mm_Horizontal, symbol Device:R_US
- removed R3, R4: 200, Resistor_THT:R_Axial_DIN0207_L6.3mm_D2.5mm_P10.16mm_Horizontal, symbol Device:R_US
- removed U1, U2: CNY70, Connector_PinHeader_2.54mm:PinHeader_1x04_P2.54mm_Vertical, symbol Sensor_Proximity:CNY70
- added D?: D, symbol Device:D
- added J?: Screw_Terminal_01x02, symbol Connector:Screw_Terminal_01x02
- added SensoresPISO1, SensoresPISO2: Conn_01x04, Connector_PinSocket_2.54mm:PinSocket_1x04_P2.54mm_Vertical, symbol Connector_Generic:Conn_01x04
Connections:
- net +5V: now also A2.10 (A1), A2.9 (A0), SensoresPISO1.1 (Pin_1), SensoresPISO2.1 (Pin_1)
- net Earth: now also J?.2 (Pin_2)
- net GND: now also SensoresPISO1.3 (Pin_3), SensoresPISO2.3 (Pin_3)
- net SENSOR DE PISO 1: now also SensoresPISO1.4 (Pin_4)
- net SENSOR DE PISO 2: now also SensoresPISO2.4 (Pin_4)
- net at D2.2 (A), SW1.2 (B): now also J?.1 (Pin_1)
- net at SW1.1 (A): now also D?.2 (A)
- no-connect marks 0 -> 2
Other:
- moved on the sheet: D2, R1, SW2

Commit message: Esquematico terminado y esquemas del step down y step up
Parts:
- added J?: Screw_Terminal_01x02, symbol Connector:Screw_Terminal_01x02
- added U?: ~, symbol Mt3608:LM2596
- added U?: ~, symbol Mt3608:mt3608
Connections:
- net Earth: now also U?.VIN-, U?.VIN-
- net GND: now also U?.VOUT-
- net STEP DOWN: now reaches D?.1 (K)
- net STEP DOWN: now also U?.VIN+, U?.VIN+
- net VIN: now reaches A1.30 (VIN)
- net VIN: now also U?.VOUT+
- new net: J?.2 (Pin_2), U?.VOUT+
- new net: J?.1 (Pin_1), U?.VOUT-

Commit message: Huella step Down
Parts:
- U2: renamed from U?; footprint (none) -> Step Down:Step Down
- gave numbers to parts that had none: 4
Changed lines of the file:
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@@
 		(dnp no)
 		(fields_autoplaced yes)
-		(property "Reference" "U?"
+		(property "Reference" "U2"
 			(at 43.942 141.224 0)
 			(effects
@@
 			)
 		)
-		(property "Footprint" ""
+		(property "Footprint" "Step Down:Step Down"
 			(at 37.592 147.066 0)
 			(effects
@@
 			(project "Clase de Club robotica"
 				(path "/feeeb2cb-e374-40f4-b9c7-40ed321ecf02"
-					(reference "U?")
+					(reference "U2")
 					(unit 1)
 				)
@@
 		(dnp no)
 		(fields_autoplaced yes)
-		(property "Reference" "U?"
+		(property "Reference" "U1"
 			(at 43.688 130.048 0)
 			(effects
@@
 			(project "Clase de Club robotica"
 				(path "/feeeb2cb-e374-40f4-b9c7-40ed321ecf02"
-					(reference "U?")
+					(reference "U1")
 					(unit 1)
 				)
@@
 		(dnp no)
 		(fields_autoplaced yes)
-		(property "Reference" "D?"
+		(property "Reference" "D1"
 			(at 69.342 87.122 0)
 			(effects
@@
 			(project "Clase de Club robotica"
 				(path "/feeeb2cb-e374-40f4-b9c7-40ed321ecf02"
-					(reference "D?")
+					(reference "D1")
 					(unit 1)
 				)
@@
 		(dnp no)
 		(fields_autoplaced yes)
-		(property "Reference" "J?"
+		(property "Reference" "J6"
 			(at 102.87 93.4719 0)
 			(effects
@@
 			(project "Clase de Club robotica"
 				(path "/feeeb2cb-e374-40f4-b9c7-40ed321ecf02"
-					(reference "J?")
+					(reference "J6")
 					(unit 1)
 				)
@@
 		(dnp no)
 		(fields_autoplaced yes)
-		(property "Reference" "J?"
+		(property "Reference" "J2"
 			(at 25.146 129.286 0)
 			(effects
@@
 			(project "Clase de Club robotica"
 				(path "/feeeb2cb-e374-40f4-b9c7-40ed321ecf02"
-					(reference "J?")
-					(unit 1)
-				)
+					(reference "J2")
+					(unit 1)
+				)

Commit message: No se
Parts:
- removed J5: Ultrasonico 4, Connector_PinHeader_2.54mm:PinHeader_1x04_P2.54mm_Vertical, symbol Connector_Generic:Conn_01x04
Connections:
- net ECHO 4 is gone; now on net AIN1 MONSTER SHIELD: A1.15 (D12)
- net TRIG 4 is gone; now on net AIN2 MONSTER SHIELD: A1.16 (D13)
- net AIN1 MONSTER SHIELD: no longer A1.2 (D0/RX)
- net AIN2 MONSTER SHIELD: no longer A1.1 (D1/TX)
- net BOTON : now also A1.21 (A2)
- net ECHO 1: now also A1.10 (D7); no longer A1.9 (D6)
- net TRIG 1: now also A1.9 (D6); no longer A1.10 (D7)
Other:
- moved on the sheet: A1, A2, D1, D2, J1, J2, J3, J4, J6, R1, SW1, SW2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

Commit message: Quedan 4 puentes
Parts:
- added SensoresPISO3: Conn_01x04, Connector_PinSocket_2.54mm:PinSocket_1x04_P2.54mm_Vertical, symbol Connector_Generic:Conn_01x04
Connections:
- net +5V: now also SensoresPISO3.1 (Pin_1)
- net BOTON : now also A1.22 (A3); no longer A1.21 (A2)
- net GND: now also SensoresPISO3.3 (Pin_3)
- net PWM B MONSTER SHIELD: now also A1.25 (A6); no longer A1.8 (D5)
- net SENSOR DE PISO 3: now reaches A1.26 (A7)
- net SENSOR DE PISO 3: now also SensoresPISO3.4 (Pin_4)
- no-connect marks 2 -> 3

Commit message: 4 puentes
Connections:
- net AIN1 MONSTER SHIELD: now also A1.25 (A6); no longer A1.15 (D12)
- net PWM B MONSTER SHIELD: now also A1.24 (A5); no longer A1.25 (A6)
Changed lines of the file:
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@@
 	(global_label "AIN1 MONSTER SHIELD"
 		(shape input)
-		(at 158.75 73.66 180)
-		(fields_autoplaced yes)
-		(effects
-			(font
-				(size 1.27 1.27)
-			)
-			(justify right)
-		)
-		(property "Intersheetrefs" "${INTERSHEET_REFS}"
-			(at 134.2958 73.66 0)
-			(effects
-				(font
-					(size 1.27 1.27)
-				)
-				(justify right)
+		(at 184.15 73.66 0)
+		(fields_autoplaced yes)
+		(effects
+			(font
+				(size 1.27 1.27)
+			)
+			(justify left)
+		)
+		(property "Intersheetrefs" "${INTERSHEET_REFS}"
+			(at 208.6042 73.66 0)
+			(effects
+				(font
+					(size 1.27 1.27)
+				)
+				(justify left)
 				(hide yes)
 			)
@@
 	(global_label "PWM B MONSTER SHIELD"
 		(shape input)
-		(at 184.15 73.66 0)
+		(at 184.15 71.12 0)
 		(fields_autoplaced yes)
 		(effects
@@
 		)
 		(property "Intersheetrefs" "${INTERSHEET_REFS}"
-			(at 210.7812 73.66 0)
-			(effects
-				(font
+			(at 210.7812 71.12 0)
+			(effects
+				(font
