File: Electronica/PCB/Clase de Club robotica/Clase de Club robotica.kicad_sch (KiCad schematic)
At the start: 17 parts, among them J1 Ultrasonico 1, J2 Screw_Terminal_01x02, J3 Ultrasonico 2, J4 Ultrasonico 3, J5 Ultrasonico 4, J6 Screw_Terminal_01x02, SW1 SW_SPST, SW2 SW_Push

Commit message: Placa hoy le pregunto a prieto del diseño
Parts:
- removed J5: Ultrasonico 4, Connector_PinHeader_2.54mm:PinHeader_1x04_P2.54mm_Vertical, symbol Connector_Generic:Conn_01x04
- added SensoresPISO3: Conn_01x04, Connector_PinSocket_2.54mm:PinSocket_1x04_P2.54mm_Vertical, symbol Connector_Generic:Conn_01x04
- D1: footprint (none) -> Diode_THT:D_5W_P10.16mm_Horizontal
- J2: footprint (none) -> TerminalBlock:TerminalBlock_bornier-2_P5.08mm
- J6: footprint (none) -> Connector_PinSocket_2.54mm:PinSocket_1x02_P2.54mm_Vertical
- U1: footprint (none) -> misc_footprints:MT3608_module
Connections:
- net TRIG 4 is gone; now on net AIN2 MONSTER SHIELD: A1.16 (D13)
- net +5V: now also SensoresPISO3.1 (Pin_1)
- net AIN1 MONSTER SHIELD: now also A1.25 (A6); no longer A1.2 (D0/RX)
- net AIN2 MONSTER SHIELD: no longer A1.1 (D1/TX)
- net BOTON : now also A1.22 (A3)
- net GND: now also SensoresPISO3.3 (Pin_3)
- net PWM B MONSTER SHIELD: now also A1.24 (A5); no longer A1.8 (D5)
- net SENSOR DE PISO 3: now reaches A1.26 (A7)
- net SENSOR DE PISO 3: now also SensoresPISO3.4 (Pin_4)
- net ECHO 4: no longer names the net of A1.15 (D12)
- no-connect marks 2 -> 3
Other:
- moved on the sheet: A1, A2, D1, D2, J1, J2, J3, J4, J6, R1, SW1, SW2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
