File: Electronica/PCB/PCB ROBOTICA V3/_autosave-PCB ROBOTICA V3.kicad_sch (KiCad schematic)
At the start: 13 parts, among them J1 Ultrasonico 1, J2 Screw_Terminal_01x02, J3 Ultrasonico 2, J4 Ultrasonico 3, J5 Conn_02x05_Counter_Clockwise, J6 Screw_Terminal_01x02

Commit message: Pcb terminada
Parts:
- gave numbers to parts that had none: 1
Changed lines of the file:
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@@
 		(dnp no)
 		(fields_autoplaced yes)
-		(property "Reference" "D?"
+		(property "Reference" "D1"
 			(at 240.03 15.24 0)
 			(effects
@@
 			(project "PCB ROBOTICA V3"
 				(path "/feeeb2cb-e374-40f4-b9c7-40ed321ecf02"
-					(reference "D?")
+					(reference "D1")
 					(unit 1)
 				)
