File: Electronica/PCB/PCB de botones V1/PCB de botones V1.kicad_pcb (KiCad board)
At the start: 2 copper layers, 80.3 x 28.4 mm, 14 parts, among them J2 Conn_02x05_Counter_Clockwise, SW2 SW_Push, SW4 SW_Push, SW9 SW_SPST

Commit message: .
Other:
- board text added: "AH y otra cosa, creo que quedaria mejor si este agujero de sujecion queda por afuera como el otro"
- board text added: "Acordate de separar los pines del switch"
Changed lines of the file:
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@@
 		)
+	)
+	(gr_line
+		(start 152.7 71.5)
+		(end 156.15 71.5)
+		(stroke
+			(width 0.2)
+			(type default)
+		)
+		(layer "F.Cu")
+	)
+	(gr_line
+		(start 223.95 103.75)
+		(end 221.75 102.1)
+		(stroke
+			(width 0.2)
+			(type default)
+		)
+		(layer "F.Cu")
+	)
+	(gr_line
+		(start 154.7 66.85)
+		(end 154.75 73.1)
+		(stroke
+			(width 0.2)
+			(type default)
+		)
+		(layer "F.Cu")
+	)
+	(gr_line
+		(start 219.7 103.85)
+		(end 223.95 103.75)
+		(stroke
+			(width 0.2)
+			(type default)
+		)
+		(layer "F.Cu")
+	)
+	(gr_line
+		(start 221.7 108.6)
+		(end 221.75 102.1)
+		(stroke
+			(width 0.2)
+			(type default)
+		)
+		(layer "F.Cu")
+	)
+	(gr_line
+		(start 221.75 102.1)
+		(end 219.7 103.85)
+		(stroke
+			(width 0.2)
+			(type default)
+		)
+		(layer "F.Cu")
+	)
+	(gr_line
+		(start 154.75 73.1)
+		(end 152.7 71.5)
+		(stroke
+			(width 0.2)
+			(type default)
+		)
+		(layer "F.Cu")
+	)
+	(gr_line
+		(start 156.15 71.5)
+		(end 154.75 73.1)
+		(stroke
+			(width 0.2)
+			(type default)
+		)
+		(layer "F.Cu")
 	)
 	(gr_rect
@@
 		(layer "Edge.Cuts")
 	)
+	(gr_text "Acordate de separar los pines del switch"
+		(at 208.65 111.45 0)
+		(layer "F.Cu")
+		(effects
+			(font
+				(size 1.5 1.5)
+				(thickness 0.3)
+				(bold yes)
+			)
+			(justify left bottom)
+		)
+	)
+	(gr_text "AH y otra cosa, creo que quedaria mejor si\neste agujero de sujecion queda por afuera como el otro"
+		(at 150.25 65.7 0)
+		(layer "F.Cu")
+		(effects
+			(font
+				(size 1.5 1.5)
+				(thickness 0.3)
+				(bold yes)
+			)
+			(justify left bottom)
+		)
+	)
 	(gr_text "BETO BTN V1\n"

Commit message: pcb de leds
Parts:
- removed D10, D3, D7, D8, D9: LED, LED_THT:LED_D5.0mm
- removed J2: Conn_02x05_Counter_Clockwise, Connector_IDC:IDC-Header_2x05_P2.54mm_Vertical
- removed R10, R7, R8, R9: R_US, Resistor_THT:R_Axial_DIN0207_L6.3mm_D2.5mm_P10.16mm_Horizontal
- removed SW2, SW4: SW_Push, Button_Switch_THT:SW_PUSH_6mm
- removed SW9: SW_SPST, Button_Switch_THT:SW_Slide_SPDT_Straight_CK_OS102011MS2Q
- added BTN 1: SW_Push, Button_Switch_THT:SW_PUSH_6mm, F.Cu at (191.4, 80.1)
- added BTN 2: SW_Push, Button_Switch_THT:SW_PUSH_6mm, F.Cu at (198.1, 94.2)
- added IDC 1: IDC Placa Botones, Connector_IDC:IDC-Header_2x05_P2.54mm_Horizontal, F.Cu at (181.4, 92.3)
- added Led 1: LED, LED_THT:LED_D5.0mm, F.Cu at (215.0, 83.2)
- added Led 2: LED, LED_THT:LED_D5.0mm, F.Cu at (207.8, 83.2)
- added Led 3: LED, LED_THT:LED_D5.0mm, F.Cu at (215.0, 92.2)
- added Led 4: LED, LED_THT:LED_D5.0mm, F.Cu at (207.8, 92.2)
- added R1: R_US, Resistor_THT:R_Axial_DIN0207_L6.3mm_D2.5mm_P10.16mm_Horizontal, F.Cu at (231.7, 81.5)
- added R2: R_US, Resistor_THT:R_Axial_DIN0207_L6.3mm_D2.5mm_P10.16mm_Horizontal, F.Cu at (231.7, 86.1)
- added R4: R_US, Resistor_THT:R_Axial_DIN0207_L6.3mm_D2.5mm_P10.16mm_Horizontal, F.Cu at (231.7, 94.8)
- R3: moved to F.Cu
- moved R3 80.9 mm to (231.7, 90.5), turned to 180 degrees
Routing:
- net Net-(D7-A): track 88.2 -> 0.00 mm, vias 1 -> 0
- net Net-(D10-A): track 86.7 -> 0.00 mm, vias 1 -> 0
- net LED3: track 0.00 -> 58.0 mm
- net Net-(D9-A): track 55.5 -> 0.00 mm, vias 1 -> 0
- net LED4: track 0.00 -> 55.1 mm
- net LED2: track 0.00 -> 44.0 mm
- net Net-(D8-A): track 42.8 -> 0.00 mm, vias 1 -> 0
- net LED1: track 0.00 -> 42.4 mm
- net Net-(J2-Pin_7): track 37.0 -> 0.00 mm, vias 1 -> 0
- net Net-(D3-K): track 39.7 -> 8.28 mm
- net Net-(D3-A): track 27.1 -> 0.00 mm, vias 1 -> 0
- net Net-(D9-K): track 25.4 -> 0.00 mm
- net BTN1: track 0.00 -> 23.7 mm
- net BTN2: track 0.00 -> 21.1 mm
- net Net-(J2-Pin_5): track 21.1 -> 0.00 mm, vias 1 -> 0
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- added copper zone on F.Cu, net GND
Other:
- board size 80.3 x 28.4 mm -> 67.7 x 30.9 mm
- board text removed: "AH y otra cosa, creo que quedaria mejor si este agujero de sujecion queda por afuera como el otro"
- board text removed: "Acordate de separar los pines del switch"
- board text removed: "BETO BTN V1"

Commit message: botones
Parts:
- moved R3 1.66 mm to (230.0, 90.1)
- moved R2 1.66 mm to (230.0, 85.7)
- moved R4 1.66 mm to (230.0, 94.5)
- moved R1 1.59 mm to (230.1, 81.3)
Routing:
- net GND: track 98.4 -> 104.8 mm
- net Net-(D4-K): track 16.3 -> 14.5 mm
- net Net-(D2-K): track 16.6 -> 15.2 mm
- net Net-(D1-K): track 8.20 -> 6.77 mm
- net Net-(D3-K): track 8.28 -> 7.03 mm
Other:
- board size 67.7 x 30.9 mm -> 73.5 x 32.3 mm
Changed lines of the file:
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@@
 	(footprint "Resistor_THT:R_Axial_DIN0207_L6.3mm_D2.5mm_P10.16mm_Horizontal"
 		(layer "F.Cu")
-		(at 231.66 90.47 180)
+		(at 230.04 90.1 180)
 		(descr "Resistor, Axial_DIN0207 series, Axial, Horizontal, pin pitch=10.16mm, 0.25W = 1/4W, length*diameter=6.3*2.5mm^2, http://cdn-reichelt.de/documents/datenblatt/B400/1_4W%23YAG.pdf")
 		(tags "Resistor Axial_DIN0207 series Axial Horizontal pin pitch 10.16mm 0.25W = 1/4W length 6.3mm diameter 2.5mm")
@@
 	(footprint "Resistor_THT:R_Axial_DIN0207_L6.3mm_D2.5mm_P10.16mm_Horizontal"
 		(layer "F.Cu")
-		(at 231.66 81.49 180)
+		(at 230.08 81.34 180)
 		(descr "Resistor, Axial_DIN0207 series, Axial, Horizontal, pin pitch=10.16mm, 0.25W = 1/4W, length*diameter=6.3*2.5mm^2, http://cdn-reichelt.de/documents/datenblatt/B400/1_4W%23YAG.pdf")
 		(tags "Resistor Axial_DIN0207 series Axial Horizontal pin pitch 10.16mm 0.25W = 1/4W length 6.3mm diameter 2.5mm")
@@
 	(footprint "Resistor_THT:R_Axial_DIN0207_L6.3mm_D2.5mm_P10.16mm_Horizontal"
 		(layer "F.Cu")
-		(at 231.66 94.85 180)
+		(at 230.04 94.48 180)
 		(descr "Resistor, Axial_DIN0207 series, Axial, Horizontal, pin pitch=10.16mm, 0.25W = 1/4W, length*diameter=6.3*2.5mm^2, http://cdn-reichelt.de/documents/datenblatt/B400/1_4W%23YAG.pdf")
 		(tags "Resistor Axial_DIN0207 series Axial Horizontal pin pitch 10.16mm 0.25W = 1/4W length 6.3mm diameter 2.5mm")
@@
 	(footprint "Resistor_THT:R_Axial_DIN0207_L6.3mm_D2.5mm_P10.16mm_Horizontal"
 		(layer "F.Cu")
-		(at 231.66 86.1 180)
+		(at 230.04 85.73 180)
 		(descr "Resistor, Axial_DIN0207 series, Axial, Horizontal, pin pitch=10.16mm, 0.25W = 1/4W, length*diameter=6.3*2.5mm^2, http://cdn-reichelt.de/documents/datenblatt/B400/1_4W%23YAG.pdf")
 		(tags "Resistor Axial_DIN0207 series Axial Horizontal pin pitch 10.16mm 0.25W = 1/4W length 6.3mm diameter 2.5mm")
@@
 		)
 		(property "Value" "SW_Push"
-			(at 3.75 6.7 360)
+			(at 3.75 6.7 0)
 			(layer "F.Fab")
 			(effects
@@
 		)
 		(fp_text user "${REFERENCE}"
-			(at 3.25 2.25 360)
+			(at 3.25 2.25 0)
 			(layer "F.Fab")
 			(effects
@@
 		)
 		(fp_text user "${REFERENCE}"
-			(at 8.83 5.08 270)
+			(at 8.83 5.08 -90)
 			(layer "F.Fab")
 			(effects
@@
 	)
 	(gr_rect
-		(start 166.18 73.5)
-		(end 233.88 104.44)
+		(start 162.53 73.5)
+		(end 236.07 105.8)
 		(stroke
 			(width 0.05)
@@
 	)
 	(via
-		(at 168.87 101.1)
+		(at 165.14 102.68)
 		(size 5)
 		(drill 3.2)
@@
 	)
 	(via
-		(at 230.82 76.36)
+		(at 232.99 76.84)
 		(size 5)
 		(drill 3.2)
@@
 	)
 	(segment
-		(start 221.5 83.16)
-		(end 221.5 81.49)
+		(start 219.92 81.34)
+		(end 214.97 81.34)
 		(width 1)
 		(layer "B.Cu")
@@
 	)
 	(segment
-		(start 214.97 83.16)
-		(end 221.5 83.16)
+		(start 214.97 81.34)
+		(end 214.97 83.16)
 		(width 1)
 		(layer "B.Cu")
@@
 	)
 	(segment
-		(start 221.5 92.22)
-		(end 221.5 90.47)
+		(start 214.97 90.1)
+		(end 214.97 92.22)
 		(width 1)
 		(layer "B.Cu")
@@
 	)
 	(segment
-		(start 214.97 92.22)
-		(end 221.5 92.22)
+		(start 219.88 90.1)
+		(end 214.97 90.1)
 		(width 1)
 		(layer "B.Cu")
@@
 	)
 	(segment
-		(start 185.76 97.72)
-		(end 185.87 97.83)
-		(width 1)
-		(layer "F.Cu")
-		(net 3)
-	)
-	(segment
-		(start 185.76 92.35)
-		(end 185.76 97.72)
-		(width 1)
-		(layer "F.Cu")
-		(net 3)
-	)
-	(segment
-		(start 185.87 97.83)
-		(end 228.68 97.83)
+		(start 189.55 92.35)
+		(end 185.76 92.35)
 		(width 1)
 		(layer "F.Cu")
@@
 	)
 	(segment
-		(start 194.31 89.77)
-		(end 194.35 89.73)
+		(start 189.99 91.91)
+		(end 189.55 92.35)
 		(width 1)
 		(layer "F.Cu")
@@
 	)
 	(segment
-		(start 194.31 97.87)
-		(end 194.31 89.77)
+		(start 185.83 102.14)
+		(end 185.76 102.07)
 		(width 1)
 		(layer "F.Cu")
@@
 	)
 	(segment
-		(start 194.33 97.89)
-		(end 194.31 97.87)
+		(start 185.76 102.07)
+		(end 185.76 92.35)
 		(width 1)
 		(layer "F.Cu")
@@
 	)
 	(via
-		(at 194.35 89.73)
+		(at 185.83 102.14)
 		(size 0.6)
 		(drill 0.3)
@@
 	)
 	(via
-		(at 228.68 97.83)
+		(at 185.76 92.35)
 		(size 0.6)
 		(drill 0.3)
@@
 	)
 	(via
-		(at 185.76 92.35)
+		(at 189.99 91.91)
 		(size 0.6)
 		(drill 0.3)
@@
 	)
 	(segment
-		(start 231.66 97.82)
-		(end 231.67 97.83)
+		(start 189.99 91.34)
+		(end 191.6 89.73)
 		(width 1)
 		(layer "B.Cu")
@@
 	)
 	(segment
-		(start 231.67 97.83)
-		(end 228.68 97.83)
+		(start 189.99 91.91)
+		(end 189.99 91.34)
 		(width 1)
 		(layer "B.Cu")
@@
 	)
 	(segment
-		(start 231.66 81.49)
-		(end 231.66 86.1)
+		(start 230.04 81.12)
+		(end 230.04 85.73)
 		(width 1)
 		(layer "B.Cu")
@@
 	)
 	(segment
-		(start 231.66 86.1)
-		(end 231.66 90.47)
+		(start 230.04 85.73)
+		(end 230.04 90.1)
 		(width 1)
 		(layer "B.Cu")
@@
 	)
 	(segment
+		(start 185.83 102.14)
+		(end 230.04 102.14)
+		(width 1)
+		(layer "B.Cu")
+		(net 3)
+	)
+	(segment
 		(start 181.3975 92.34)
 		(end 185.75 92.34)
@@
 	)
 	(segment
-		(start 231.66 94.85)
-		(end 231.66 97.82)
+		(start 230.04 90.1)
+		(end 230.04 94.48)
 		(width 1)
 		(layer "B.Cu")
@@
 	)
 	(segment
-		(start 231.66 90.47)
-		(end 231.66 94.85)
+		(start 230.04 94.48)
+		(end 230.04 102.14)
 		(width 1)
 		(layer "B.Cu")
@@
 	)
 	(segment
-		(start 207.82 86.1)
-		(end 221.5 86.1)
+		(start 219.88 85.73)
+		(end 208.19 85.73)
+		(width 1)
+		(layer "B.Cu")
+		(net 6)
+	)
+	(segment
+		(start 208.19 85.73)
+		(end 207.82 86.1)
 		(width 1)
 		(layer "B.Cu")
@@
 	)
 	(segment
+		(start 207.92 94.48)
+		(end 219.88 94.48)
+		(width 1)
+		(layer "B.Cu")
+		(net 8)
+	)
+	(segment
 		(start 207.82 92.22)
-		(end 207.82 94.85)
+		(end 207.82 94.58)
 		(width 1)
 		(layer "B.Cu")
@@
 	)
 	(segment
-		(start 207.82 94.85)
-		(end 221.5 94.85)
+		(start 207.82 94.58)
+		(end 207.92 94.48)
 		(width 1)
 		(layer "B.Cu")
@@
 		(polygon
 			(pts
-				(xy 166.13 72.67) (xy 166.18 104.52) (xy 233.73 104.52) (xy 233.97 73.47) (xy 166.42 73.52) (xy 166.287555 72.508416)
+				(xy 162.55 73.27) (xy 162.5 105.38) (xy 236.28 105.73) (xy 236.4 73.57) (xy 166.42 73.51) (xy 166.27 73.51)
 			)
 		)

Commit message: Listo PCB Botones
Parts:
- added ?: , , F.Cu at (168.8, 100.3)
- added ?: , , F.Cu at (232.8, 76.8)
- moved IDC 1 3.55 mm to (184.9, 92.3)
Routing:
- net BTN2: track 21.1 -> 17.4 mm
- net LED2: track 44.0 -> 40.4 mm
- net LED4: track 55.1 -> 51.9 mm
- net LED3: track 58.0 -> 54.8 mm
- net BTN1: track 23.7 -> 20.7 mm
- net LED1: track 42.4 -> 39.7 mm
- net GND: track 104.8 -> 103.3 mm, vias 3 -> 4
- net Net-(D2-K): track 15.2 -> 14.6 mm
- net (no net): vias 2 -> 0
- removed copper zone on F.Cu, net GND
Other:
- board size 73.5 x 32.3 mm -> 70.5 x 30.1 mm

Commit message: Codigo nuevo sin terminar
Parts:
- added ?: , , F.Cu at (167.8, 76.4)
- added ?: , , F.Cu at (234.2, 100.6)
- moved ? 1.50 mm to (234.2, 76.4)
- moved ? 1.09 mm to (167.8, 100.6)
Routing:
- net GND: track 103.3 -> 108.8 mm
- net LED2: track 40.4 -> 41.6 mm
- net LED3: track 54.8 -> 55.6 mm
- net LED4: track 51.9 -> 52.4 mm
Other:
- board size 70.5 x 30.1 mm -> 72.5 x 30.1 mm
