File: Electronica/PCB/PCB de Sensores V1/PCB de Sensores V1.kicad_sch (KiCad schematic)
At the start: 10 parts, among them J1 Conn_02x08_Odd_Even, J2 Conexion Sensores, U1 ULTRASONICO1, U2 ULTRASONICO2, U3 ULTRASONICO3, U4 ULTRASONICO4, U5 ULTRASONICO5

Commit message: SELIGRAFIA
Connections:
- net +5V: now also J2.10 (Pin_10); no longer J2.15 (Pin_15)
- net CNY 1: now also J2.16 (Pin_16); no longer J2.9 (Pin_9)
- net CNY 2: now also J2.5 (Pin_5); no longer J2.11 (Pin_11)
- net CNY 3: now also J2.2 (Pin_2); no longer J2.13 (Pin_13)
- net ECHO 1: now also J2.15 (Pin_15); no longer J2.7 (Pin_7)
- net ECHO 3: now also J2.12 (Pin_12); no longer J2.2 (Pin_2)
- net ECHO 4: now also J2.6 (Pin_6); no longer J2.8 (Pin_8)
- net ECHO 5: now also J2.7 (Pin_7); no longer J2.12 (Pin_12)
- net GND: now also J2.11 (Pin_11); no longer J2.16 (Pin_16)
- net TRIG 1: now also J2.13 (Pin_13); no longer J2.5 (Pin_5)
- net TRIG 3: now also J2.14 (Pin_14); no longer J2.4 (Pin_4)
- net TRIG 4: now also J2.8 (Pin_8); no longer J2.10 (Pin_10)
- net TRIG 5: now also J2.9 (Pin_9); no longer J2.14 (Pin_14)
Other:
- note added: "AHI LO HICE, TERMINA LA PLACA"

Commit message: Codigo nuevo sin terminar
Parts:
- removed J2: Conexion Sensores, Connector_PinHeader_2.54mm:PinHeader_2x08_P2.54mm_Horizontal, symbol Connector_Generic:Conn_02x08_Odd_Even
Other:
- note removed: "AHI LO HICE, TERMINA LA PLACA"
- note removed: "Te dejo las conexiones que quedaron en la placa principal para que las corrijas"

Commit message: ?
Parts:
- J1: value Conn_02x08_Odd_Even -> Conexion Sensores
Connections:
- net +5V: now also J1.15 (Pin_15); no longer J1.10 (Pin_10)
- net GND: now also J1.16 (Pin_16); no longer J1.11 (Pin_11)
- net TRIG 3: now reaches J1.4 (Pin_4)
- net TRIG 3: now also U3.3 (Pin_3)
- net CNY1 renamed CNY 1
- net CNY 1: now also J1.9 (Pin_9); no longer J1.16 (Pin_16)
- net CNY2 renamed CNY 2
- net CNY 2: now also J1.11 (Pin_11); no longer J1.5 (Pin_5)
- net CNY3 renamed CNY 3
- net CNY 3: now also J1.13 (Pin_13); no longer J1.2 (Pin_2)
- net ECHO1 renamed ECHO 1
- net ECHO 1: now also J1.7 (Pin_7); no longer J1.15 (Pin_15)
- net ECHO2 renamed ECHO 2
- net ECHO3 renamed ECHO 3
- net ECHO 3: now also J1.2 (Pin_2); no longer J1.12 (Pin_12)
- net ECHO4: no longer names the net of J1.6 (Pin_6)
- net ECHO4: no longer U4.2 (Pin_2)
- net ECHO5 renamed ECHO 5
- net ECHO 5: now also J1.12 (Pin_12); no longer J1.7 (Pin_7)
- net TRIG1 renamed TRIG 1
- net TRIG 1: now also J1.5 (Pin_5); no longer J1.13 (Pin_13)
- net TRIG2 renamed TRIG 2
- net TRIG3 renamed TRIG 5
- net TRIG 5: now also U5.3 (Pin_3); no longer U3.3 (Pin_3)
- net TRIG4 renamed ECHO 4
- net ECHO 4: now also U4.2 (Pin_2); no longer U4.3 (Pin_3)
- removed net TRIG5: J1.9 (Pin_9), U5.3 (Pin_3)
- new net TRIG 4: J1.10 (Pin_10), U4.3 (Pin_3)

Commit message: pcb sensores corregida
Tonto el que lee
Parts:
- U3: footprint Connector_PinHeader_2.54mm:PinHeader_1x04_P2.54mm_Horizontal -> Connector_PinHeader_2.54mm:PinHeader_1x04_P2.54mm_Vertical
- U5: footprint Connector_PinHeader_2.54mm:PinHeader_1x04_P2.54mm_Vertical -> Connector_PinHeader_2.54mm:PinHeader_1x04_P2.54mm_Horizontal
Changed lines of the file:
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@@
 			)
 		)
-		(property "Footprint" "Connector_PinHeader_2.54mm:PinHeader_1x04_P2.54mm_Horizontal"
+		(property "Footprint" "Connector_PinHeader_2.54mm:PinHeader_1x04_P2.54mm_Vertical"
 			(at 55.88 45.72 0)
 			(effects
@@
 			)
 		)
-		(property "Footprint" "Connector_PinHeader_2.54mm:PinHeader_1x04_P2.54mm_Vertical"
+		(property "Footprint" "Connector_PinHeader_2.54mm:PinHeader_1x04_P2.54mm_Horizontal"
 			(at 30.48 39.37 0)
 			(effects
