File: Electronica/PCB/PCB Principal V6/PCB Principal V6.kicad_pcb (KiCad board)
At the start: 2 copper layers, 139.1 x 70 mm, 18 parts, among them J1 Conexion Sensores, J12 TP, J2 Power Monster, J3 On/Off General, J4 Power Input 2, J5 IDC Placa Botones, J6 Power Input 1, J7 Conn_01x01_Pin, J8 Conn_01x01_Pin, SW1 On/Off Motores

Commit message: ,
Parts:
- added LM1: LM2596_OK, StepDown:StepDown, F.Cu at (39.2, 159.2)
- moved A1 139.0 mm to (52.8, 140.7)
- moved J2 123.4 mm to (105.2, 161.2)
- moved J3 123.4 mm to (105.2, 170.2)
- moved R1 118.0 mm to (103.5, 176.3)
- moved R2 118.0 mm to (103.5, 179.5)
- moved SW1 117.1 mm to (74.3, 174.3)
- moved J5 108.7 mm to (88.4, 159.0)
- moved J1 108.0 mm to (72.4, 138.5)
- moved J4 108.0 mm to (91.2, 141.3)
- moved J6 108.0 mm to (91.2, 151.5)
- moved D1 106.6 mm to (87.9, 173.6)
- moved D2 106.6 mm to (87.9, 177.8)
- moved D3 104.3 mm to (72.6, 160.3)
- moved D4 104.3 mm to (80.1, 160.3)
- moved J12 100.9 mm to (105.9, 138.5)
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
Commit message: PCB CHERNIAK TERMINAR
TONTO EL QUE LEE
Parts:
- moved LM1 224.9 mm to (242.6, 63.2)
- moved SW1 195.0 mm to (250.8, 91.5)
- moved J5 194.4 mm to (240.5, 37.9), turned to 90 degrees
- moved A1 182.3 mm to (208.3, 45.7)
- moved D3 182.2 mm to (239.8, 88.0)
- moved R1 175.5 mm to (254.6, 87.1), turned to 180 degrees
- moved J1 174.7 mm to (215.1, 37.7), turned to 90 degrees
- moved J3 146.3 mm to (228.1, 90.8)
- moved A2 141.6 mm to (200.9, 53.6), turned to -90 degrees
- moved D1 138.8 mm to (140.7, 45.2), turned to 180 degrees
- moved D2 137.9 mm to (140.7, 50.4), turned to 180 degrees
- moved J6 128.3 mm to (133.1, 30.2), turned to -90 degrees
- moved J4 122.7 mm to (143.3, 30.2), turned to -90 degrees
- moved R2 102.8 mm to (137.7, 82.5)
- moved D4 94.3 mm to (140.6, 88.0)
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Routing:
- net (no net): vias 0 -> 2

Commit message: pcb terminar?
TONTO EL QUE LEE
Parts:
- removed J12: TP, Connector_PinHeader_2.54mm:PinHeader_1x05_P2.54mm_Vertical
- added J10: Conn_01x01, Connector_PinHeader_2.54mm:PinHeader_1x01_P2.54mm_Vertical, F.Cu at (150.7, 67.6)
- added J9: Conn_01x01, Connector_PinHeader_2.54mm:PinHeader_1x01_P2.54mm_Vertical, F.Cu at (154.9, 67.7)
- A2: moved to B.Cu
- J7, J8: value Conn_01x01_Pin -> Conn_01x01
- moved SW1 109.8 mm to (141.0, 91.7)
- moved J3 75.6 mm to (152.5, 91.3)
- moved D1 43.3 mm to (159.2, 84.3)
- moved J7 38.8 mm to (154.2, 31.3), turned to 0 degrees
- moved A2 36.2 mm to (164.7, 51.7)
- moved D2 34.3 mm to (159.2, 79.3)
- moved J6 25.6 mm to (130.3, 55.7), turned to 0 degrees
- moved J4 16.0 mm to (137.5, 45.2), turned to 180 degrees
- moved A1 14.2 mm to (219.6, 54.3)
- moved D4 10.1 mm to (130.5, 88.2)
- moved LM1 8.14 mm to (250.7, 63.2)
- moved J5 7.44 mm to (247.9, 37.9)
- moved J1 7.13 mm to (222.2, 37.9)
- moved J8 5.00 mm to (145.4, 67.3), turned to 0 degrees
- moved J2 2.99 mm to (129.3, 78.9)
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Connections:
- J7 pad 1: +5V -> VNano
- J8 pad 1: GND -> PI+
Routing:
- net GND: track 0.00 -> 124.3 mm, vias 0 -> 2
- net MOTORES: track 0.00 -> 69.9 mm
- net PI+: track 0.00 -> 48.3 mm
- net Net-(J2-Pin_2): track 0.00 -> 33.9 mm
- net +5V: track 0.00 -> 19.3 mm
- net Net-(D4-A): track 0.00 -> 12.8 mm
- net Net-(D1-K): track 0.00 -> 12.7 mm
- net Net-(J4-Pin_2): track 0.00 -> 10.5 mm
- net BIN 2 MONSTER SHIELD: track 0.00 -> 7.57 mm
- net AIN2 MONSTER SHIELD: track 0.00 -> 7.28 mm
- net PWM B MONSTER SHIELD: track 0.00 -> 6.65 mm
- net PWM A MONSTER SHIELD: track 0.00 -> 6.65 mm
- net BIN 1 MONSTER SHIELD: track 0.00 -> 6.65 mm
- net AIN1 MONSTER SHIELD: track 0.00 -> 6.65 mm
- net Net-(D3-A): track 0.00 -> 3.93 mm

Commit message: .
Parts:
- added ?: , , F.Cu at (127.5, 28.4)
- added ?: , , F.Cu at (260.1, 91.7)
Routing:
- net (no net): vias 2 -> 0
Changed lines of the file:
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@@
 		(tags "XT60 female vertical")
 		(property "Reference" "J6"
-			(at 3.6 -5.3 360)
+			(at 3.6 -5.3 0)
 			(layer "F.SilkS")
 			(effects
@@
 		)
 		(property "Value" "Power Input 1"
-			(at 3.6 5.4 360)
+			(at 3.6 5.4 0)
 			(layer "F.Fab")
 			(effects
@@
 		)
 		(fp_text user "${REFERENCE}"
-			(at 3.6 0.05 360)
+			(at 3.6 0.05 0)
 			(layer "F.Fab")
 			(effects
@@
 		(tags "terminal block bornier2")
 		(property "Reference" "J3"
-			(at 2.54 -5.08 360)
+			(at 2.54 -5.08 0)
 			(layer "F.SilkS")
 			(effects
@@
 		)
 		(property "Value" "On/Off General"
-			(at 2.54 5.08 360)
+			(at 2.54 5.08 0)
 			(layer "F.Fab")
 			(effects
@@
 		)
 		(fp_text user "${REFERENCE}"
-			(at 2.54 0 360)
+			(at 2.54 0 0)
 			(layer "F.Fab")
 			(effects
@@
 		(tags "Resistor Axial_DIN0204 series Axial Horizontal pin pitch 7.62mm 0.167W length 3.6mm diameter 1.6mm")
 		(property "Reference" "R2"
-			(at 3.81 -1.92 360)
+			(at 3.81 -1.92 0)
 			(layer "F.SilkS")
 			(effects
@@
 		)
 		(property "Value" "220"
-			(at 3.81 1.92 360)
+			(at 3.81 1.92 0)
 			(layer "F.Fab")
 			(effects
@@
 		)
 		(fp_text user "${REFERENCE}"
-			(at 3.81 0 360)
+			(at 3.81 0 0)
 			(layer "F.Fab")
 			(effects
@@
 		)
 	)
+	(footprint ""
+		(layer "F.Cu")
+		(at 127.508 28.448)
+		(property "Reference" ""
+			(at 0 0 0)
+			(unlocked yes)
+			(layer "F.SilkS")
+			(effects
+				(font
+					(size 1.27 1.27)
+				)
+			)
+		)
+		(property "Value" ""
+			(at 0 0 0)
+			(unlocked yes)
+			(layer "F.Fab")
+			(effects
+				(font
+					(size 1.27 1.27)
+				)
+			)
+		)
+		(property "Footprint" ""
+			(at 0 0 0)
+			(unlocked yes)
+			(layer "F.Fab")
+			(hide yes)
+			(effects
+				(font
+					(size 1.27 1.27)
+				)
+			)
+		)
+		(property "Datasheet" ""
+			(at 0 0 0)
+			(unlocked yes)
+			(layer "F.Fab")
+			(hide yes)
+			(effects
+				(font
+					(size 1.27 1.27)
+				)
+			)
+		)
+		(property "Description" ""
+			(at 0 0 0)
+			(unlocked yes)
+			(layer "F.Fab")
+			(hide yes)
+			(effects
+				(font
+					(size 1.27 1.27)
+				)
+			)
+		)
+		(pad "2" thru_hole circle
+			(at 0 0 180)
+			(size 5 5)
+			(drill 3)
+			(layers "*.Cu" "*.Mask")
+			(remove_unused_layers no)
+			(pinfunction "IOREF")
+			(pintype "output")
+		)
+	)
 	(footprint "Resistor_THT:R_Axial_DIN0204_L3.6mm_D1.6mm_P7.62mm_Horizontal"
 		(layer "F.Cu")
@@
 		)
 	)
+	(footprint ""
+		(layer "F.Cu")
+		(at 260.096 91.694)
+		(property "Reference" ""
+			(at 0 0 0)
+			(unlocked yes)
+			(layer "F.SilkS")
+			(effects
+				(font
+					(size 1.27 1.27)
+				)
+			)
+		)
+		(property "Value" ""
+			(at 0 0 0)
+			(unlocked yes)
+			(layer "F.Fab")
+			(effects
+				(font
+					(size 1.27 1.27)
+				)
+			)
+		)
+		(property "Footprint" ""
+			(at 0 0 0)
+			(unlocked yes)
+			(layer "F.Fab")
+			(hide yes)
+			(effects
+				(font
+					(size 1.27 1.27)
+				)
+			)
+		)
+		(property "Datasheet" ""
+			(at 0 0 0)
+			(unlocked yes)
+			(layer "F.Fab")
+			(hide yes)
+			(effects
+				(font
+					(size 1.27 1.27)
+				)
+			)
+		)
+		(property "Description" ""
+			(at 0 0 0)
+			(unlocked yes)
+			(layer "F.Fab")
+			(hide yes)
+			(effects
+				(font
+					(size 1.27 1.27)
+				)
+			)
+		)
+		(pad "2" thru_hole circle
+			(at 0 0 180)
+			(size 5 5)
+			(drill 3)
+			(layers "*.Cu" "*.Mask")
+			(remove_unused_layers no)
+			(pinfunction "IOREF")
+			(pintype "output")
+		)
+	)
 	(footprint "LED_THT:LED_D5.0mm_Horizontal_O1.27mm_Z3.0mm"
 		(layer "F.Cu")
@@
 		(layer "Edge.Cuts")
 	)
-	(via
-		(at 127.7 28.4)
-		(size 5)
-		(drill 3)
-		(layers "F.Cu" "B.Cu")
-		(net 0)
-	)
-	(via
-		(at 260.09 91.28)
-		(size 5)
-		(drill 3)
-		(layers "F.Cu" "B.Cu")
-		(net 0)
-	)
 	(segment

Commit message: ?
Connections:
- A1 pad 23: LED3 -> LED2
- A1 pad 24: LED2 -> LED3
Routing:
- net LED1: track 0.00 -> 63.1 mm
- net BTN1: track 0.00 -> 51.3 mm
- net BTN2: track 0.00 -> 46.4 mm
- net LED2: track 0.00 -> 43.8 mm
Changed lines of the file:
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@@
 			)
 		)
-		(sheetname "Root")
+		(sheetname "Raíz")
 		(sheetfile "PCB Principal V6.kicad_sch")
 		(attr through_hole)
@@
 		)
 		(property ki_fp_filters "Connector*:*_1x??_*")
-		(sheetname "Root")
+		(sheetname "Raíz")
 		(sheetfile "PCB Principal V6.kicad_sch")
 		(attr through_hole)
@@
 		)
 		(property ki_fp_filters "Connector*:*_1x??_*")
-		(sheetname "Root")
+		(sheetname "Raíz")
 		(sheetfile "PCB Principal V6.kicad_sch")
 		(attr through_hole)
@@
 		)
 		(property ki_fp_filters "Connector*:*_2x??_*")
-		(sheetname "Root")
+		(sheetname "Raíz")
 		(sheetfile "PCB Principal V6.kicad_sch")
 		(attr through_hole)
@@
 		)
 		(property ki_fp_filters "LED* LED_SMD:* LED_THT:*")
-		(sheetname "Root")
+		(sheetname "Raíz")
 		(sheetfile "PCB Principal V6.kicad_sch")
 		(attr through_hole)
@@
 		)
 		(property ki_fp_filters "Connector*:*_2x??_*")
-		(sheetname "Root")
+		(sheetname "Raíz")
 		(sheetfile "PCB Principal V6.kicad_sch")
 		(attr through_hole)
@@
 		)
 		(property ki_fp_filters "TerminalBlock*:*")
-		(sheetname "Root")
+		(sheetname "Raíz")
 		(sheetfile "PCB Principal V6.kicad_sch")
 		(attr through_hole)
@@
 		)
 		(property ki_fp_filters "TerminalBlock*:*")
-		(sheetname "Root")
+		(sheetname "Raíz")
 		(sheetfile "PCB Principal V6.kicad_sch")
 		(attr through_hole)
@@
 			)
 		)
-		(sheetname "Root")
+		(sheetname "Raíz")
 		(sheetfile "PCB Principal V6.kicad_sch")
 		(attr through_hole)
@@
 		)
 		(property ki_fp_filters "Connector*:*_1x??_*")
-		(sheetname "Root")
+		(sheetname "Raíz")
 		(sheetfile "PCB Principal V6.kicad_sch")
 		(attr through_hole)
@@
 		)
 		(property ki_fp_filters "R_*")
-		(sheetname "Root")
+		(sheetname "Raíz")
 		(sheetfile "PCB Principal V6.kicad_sch")
 		(attr through_hole)
@@
 		)
 		(property ki_fp_filters "R_*")
-		(sheetname "Root")
+		(sheetname "Raíz")
 		(sheetfile "PCB Principal V6.kicad_sch")
 		(attr through_hole)
@@
 		)
 		(property ki_fp_filters "Arduino*Nano*")
-		(sheetname "Root")
+		(sheetname "Raíz")
 		(sheetfile "PCB Principal V6.kicad_sch")
 		(attr through_hole)
@@
 			(layers "*.Cu" "*.Mask")
 			(remove_unused_layers no)
-			(net 21 "LED3")
+			(net 33 "LED2")
 			(pinfunction "A4")
 			(pintype "bidirectional")
@@
 			(layers "*.Cu" "*.Mask")
 			(remove_unused_layers no)
-			(net 33 "LED2")
+			(net 21 "LED3")
 			(pinfunction "A5")
 			(pintype "bidirectional")
@@
 		)
 		(property ki_fp_filters "LED* LED_SMD:* LED_THT:*")
-		(sheetname "Root")
+		(sheetname "Raíz")
 		(sheetfile "PCB Principal V6.kicad_sch")
 		(attr through_hole)
@@
 		)
 		(property ki_fp_filters "D*DO?41*")
-		(sheetname "Root")
+		(sheetname "Raíz")
 		(sheetfile "PCB Principal V6.kicad_sch")
 		(attr through_hole)
@@
 		)
 		(property ki_fp_filters "TerminalBlock*:*")
-		(sheetname "Root")
+		(sheetname "Raíz")
 		(sheetfile "PCB Principal V6.kicad_sch")
 		(attr through_hole)
@@
 			)
 		)
-		(sheetname "Root")
+		(sheetname "Raíz")
 		(sheetfile "PCB Principal V6.kicad_sch")
 		(attr through_hole)
@@
 		)
 		(property ki_fp_filters "D*DO?41*")
-		(sheetname "Root")
+		(sheetname "Raíz")
 		(sheetfile "PCB Principal V6.kicad_sch")
 		(attr through_hole)
@@
 		)
 		(property ki_fp_filters "Connector*:*_1x??_*")
-		(sheetname "Root")
+		(sheetname "Raíz")
 		(sheetfile "PCB Principal V6.kicad_sch")
 		(attr through_hole)
@@
 		)
 		(property ki_fp_filters "Arduino*UNO*R3*")
-		(sheetname "Root")
+		(sheetname "Raíz")
 		(sheetfile "PCB Principal V6.kicad_sch")
 		(attr through_hole)
@@
 	)
 	(segment
+		(start 242.080755 78.993)
+		(end 238.833755 82.24)
+		(width 1)
+		(layer "B.Cu")
+		(net 25)
+	)
+	(segment
+		(start 255.525 37.9)
+		(end 255.525 78.993)
+		(width 1)
+		(layer "B.Cu")
+		(net 25)
+	)
+	(segment
+		(start 255.525 78.993)
+		(end 242.080755 78.993)
+		(width 1)
+		(layer "B.Cu")
+		(net 25)
+	)
+	(segment
+		(start 238.833755 82.24)
+		(end 234.85 82.24)
+		(width 1)
+		(layer "B.Cu")
+		(net 25)
+	)
+	(segment
+		(start 234.85 77.16)
+		(end 235.98137 77.16)
+		(width 1)
+		(layer "B.Cu")
+		(net 32)
+	)
+	(segment
+		(start 250.445 62.69637)
+		(end 250.445 37.9)
+		(width 1)
+		(layer "B.Cu")
+		(net 32)
+	)
+	(segment
+		(start 235.98137 77.16)
+		(end 250.445 62.69637)
+		(width 1)
+		(layer "B.Cu")
+		(net 32)
+	)
+	(segment
+		(start 244.49 37.015)
+		(end 244.49 63.488)
+		(width 1)
+		(layer "B.Cu")
+		(net 33)
+	)
+	(segment
+		(start 246.145 35.36)
+		(end 244.49 37.015)
+		(width 1)
+		(layer "B.Cu")
+		(net 33)
+	)
+	(segment
+		(start 247.905 35.36)
+		(end 246.145 35.36)
+		(width 1)
+		(layer "B.Cu")
+		(net 33)
+	)
+	(segment
+		(start 244.49 63.488)
+		(end 235.898 72.08)
+		(width 1)
+		(layer "B.Cu")
+		(net 33)
+	)
+	(segment
+		(start 235.898 72.08)
+		(end 234.85 72.08)
+		(width 1)
+		(layer "B.Cu")
+		(net 33)
+	)
+	(segment
+		(start 234.85 79.7)
+		(end 238.308 79.7)
+		(width 1)
+		(layer "B.Cu")
+		(net 36)
+	)
+	(segment
+		(start 238.308 79.7)
+		(end 252.985 65.023)
+		(width 1)
+		(layer "B.Cu")
+		(net 36)
+	)
+	(segment
+		(start 252.985 65.023)
+		(end 252.985 37.9)
+		(width 1)
+		(layer "B.Cu")
+		(net 36)
+	)
+	(segment

Commit message: .
Parts:
- J1: moved to B.Cu
- moved LM1 211.2 mm to (50.5, 130.6)
- moved D1 133.4 mm to (50.3, 161.3)
- moved D2 133.4 mm to (50.3, 156.3)
- moved J4 128.5 mm to (31.5, 117.8), turned to -90 degrees
- moved R2 128.2 mm to (35.8, 162.6), turned to -90 degrees
- moved D4 128.2 mm to (28.2, 165.5)
- moved J1 127.0 mm to (119.6, 112.8), turned to -90 degrees
- moved J6 126.6 mm to (31.5, 134.8), turned to -90 degrees
- moved J5 125.9 mm to (148.6, 115.3)
- moved SW1 125.8 mm to (41.7, 168.9)
- moved D3 125.8 mm to (141.6, 165.4)
- moved J2 125.8 mm to (30.0, 156.1)
- moved ? 125.8 mm to (28.2, 105.7)
- moved A1 125.8 mm to (120.3, 131.5)
- moved ? 125.8 mm to (160.8, 168.9)
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Connections:
- A1 pad 11: TRIG 2 -> ECHO 1
- A1 pad 14: ECHO 1 -> TRIG 2
- A1 pad 16: LED4 -> TRIG 3
- A1 pad 22: TRIG 3 -> LED2
- A1 pad 23: LED2 -> LED3
- A1 pad 24: LED3 -> LED4
- A1 pad 25: CNY 1 -> CNY 2
- A1 pad 26: CNY 2 -> CNY 1
- J1 pad 3: ECHO 2 -> TRIG 1
- J1 pad 5: TRIG 1 -> ECHO 2
Routing:
- net VNano: track 0.00 -> 172.0 mm
- net ECHO 1: track 0.00 -> 127.7 mm
- net ECHO 2: track 0.00 -> 111.8 mm
- net TRIG 1: track 0.00 -> 96.3 mm
- net TRIG 2: track 0.00 -> 79.4 mm
- net ECHO 3: track 0.00 -> 65.5 mm
- net LED1: track 63.1 -> 0.00 mm
- net TRIG 3: track 0.00 -> 60.8 mm
- net BTN1: track 51.3 -> 0.00 mm
- net BTN2: track 46.4 -> 0.00 mm
- net LED2: track 43.8 -> 0.00 mm
- net PI+: track 48.3 -> 22.8 mm
- net Net-(J2-Pin_2): track 33.9 -> 14.6 mm
- net +5V: track 19.3 -> 2.54 mm
- net MOTORES: track 69.9 -> 77.1 mm
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
Commit message: TERMINACION
-Placa Principal
-Techo de 60 Grados
-Techo Tapa
Parts:
- moved J8 135.6 mm to (42.8, 164.0)
- moved J7 115.4 mm to (59.5, 110.9)
- moved J9 112.8 mm to (65.9, 166.4), turned to 180 degrees
- moved J10 110.5 mm to (65.9, 161.7), turned to 180 degrees
- moved J5 41.0 mm to (150.1, 156.3), turned to 0 degrees
- moved D3 11.2 mm to (150.0, 172.9)
- moved ? 11.2 mm to (169.1, 176.4)
- moved R1 11.2 mm to (164.0, 172.8)
- moved J2 9.04 mm to (36.8, 162.1)
- moved J6 9.04 mm to (38.3, 140.8)
- moved A1 9.04 mm to (127.1, 137.5)
- moved A2 9.04 mm to (72.2, 134.9)
- moved D1 9.04 mm to (57.1, 167.2)
- moved D4 9.04 mm to (35.0, 171.4)
- moved ? 9.04 mm to (35.0, 111.6)
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Routing:
- net GND: track 130.6 -> 440.6 mm, vias 0 -> 6
- net +5V: track 2.54 -> 219.6 mm, vias 0 -> 2
- net MOTORES: track 77.1 -> 184.7 mm
- net CNY 1: track 0.00 -> 68.0 mm
- net CNY 2: track 0.00 -> 63.8 mm
- net LED4: track 0.00 -> 27.4 mm
- net LED3: track 0.00 -> 21.0 mm
- net LED2: track 0.00 -> 14.5 mm
- net LED1: track 0.00 -> 8.32 mm
- net BTN1: track 0.00 -> 8.32 mm
- net BTN2: track 0.00 -> 8.32 mm
- net VNano: track 172.0 -> 177.3 mm
- net PI+: track 22.8 -> 27.7 mm
