File: Electronica/PCB/PCB Principal V6/PCB Principal V6.kicad_pcb (KiCad board)
At the start: 2 copper layers, 122.4 x 78.4 mm, 20 parts, among them J1 Conexion Sensores, J11 Conn_01x04_Pin, J2 Power Monster, J3 On/Off General, J4 Power Input 2, J6 Power Input 1, J7 Placa de Botones, SW1 On/Off Motores, U1 74HC595

Commit message: nada
Parts:
- removed the ? at (98.2, 44.0)
Other:
- board text added: "CDR"
- board text removed: "CDR 2024"
Changed lines of the file:
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@@
 		)
 	)
-	(footprint ""
-		(layer "F.Cu")
-		(at 98.25 43.95)
-		(property "Reference" ""
-			(at 0 0 0)
-			(unlocked yes)
-			(layer "F.SilkS")
-			(effects
-				(font
-					(size 1.27 1.27)
-					(thickness 0.15)
-				)
-			)
-		)
-		(property "Value" ""
-			(at 0 0 0)
-			(unlocked yes)
-			(layer "F.Fab")
-			(effects
-				(font
-					(size 1.27 1.27)
-					(thickness 0.15)
-				)
-			)
-		)
-		(property "Footprint" ""
-			(at 0 0 0)
-			(unlocked yes)
-			(layer "F.Fab")
-			(hide yes)
-			(effects
-				(font
-					(size 1.27 1.27)
-					(thickness 0.15)
-				)
-			)
-		)
-		(property "Datasheet" ""
-			(at 0 0 0)
-			(unlocked yes)
-			(layer "F.Fab")
-			(hide yes)
-			(effects
-				(font
-					(size 1.27 1.27)
-					(thickness 0.15)
-				)
-			)
-		)
-		(property "Description" ""
-			(at 0 0 0)
-			(unlocked yes)
-			(layer "F.Fab")
-			(hide yes)
-			(effects
-				(font
-					(size 1.27 1.27)
-					(thickness 0.15)
-				)
-			)
-		)
-		(pad "2" thru_hole circle
-			(at 0 0 180)
-			(size 5 5)
-			(drill 3)
-			(layers "*.Cu" "*.Mask")
-			(remove_unused_layers no)
-			(pinfunction "IOREF")
-			(pintype "output")
-		)
-	)
 	(footprint "Resistor_THT:R_Axial_DIN0204_L3.6mm_D1.6mm_P7.62mm_Horizontal"
 		(layer "F.Cu")
@@
 		(layer "Edge.Cuts")
 	)
-	(gr_text "CDR \n2024"
-		(at 221.25 117.65 0)
+	(gr_text "CDR"
+		(at 224 116 0)
 		(layer "B.Cu")
 		(effects
 			(font
-				(size 3 3)
+				(size 5 5)
 				(thickness 0.4)
 			)
@@
 		)
 	)
+	(dimension
+		(type aligned)
+		(layer "F.SilkS")
+		(pts
+			(xy 228.05 122.05) (xy 228.05 43.6)
+		)
+		(height 8.95)
+		(gr_text "78,4500 mm"
+			(at 235.9 82.825 90)
+			(layer "F.SilkS")
+			(effects
+				(font
+					(size 1 1)
+					(thickness 0.1)
+				)
+			)
+		)
+		(format
+			(prefix "")
+			(suffix "")
+			(units 3)
+			(units_format 1)
+			(precision 4)
+		)
+		(style
+			(thickness 0.1)
+			(arrow_length 1.27)
+			(text_position_mode 0)
+			(extension_height 0.58642)
+			(extension_offset 0.5) keep_text_aligned)
+	)
 	(segment
