File: Electronica/PCB/PCB de Sensores V2/PCB de Sensores V2.kicad_sch (KiCad schematic)
At the start: 9 parts, among them J1 Conexion Sensores, U1 ULTRASONICO1, U2 ULTRASONICO2, U3 ULTRASONICO3, U4 ULTRASONICO4, U5 ULTRASONICO5

Commit message: PCB sensores v2 y principal v7 terminadas
Parts:
- removed C3: CNY3, Connector_PinHeader_2.54mm:PinHeader_1x04_P2.54mm_Horizontal, symbol Connector_Generic:Conn_01x04
- removed J1: Conexion Sensores, Connector_PinHeader_2.54mm:PinHeader_2x08_P2.54mm_Horizontal, symbol Connector_Generic:Conn_02x08_Odd_Even
- added J2: Conexion Sensores, Connector_PinHeader_2.54mm:PinHeader_2x08_P2.54mm_Vertical, symbol Connector_Generic:Conn_02x08_Odd_Even
- U2, U4: footprint Connector_PinHeader_2.54mm:PinHeader_1x04_P2.54mm_Horizontal -> Connector_PinHeader_2.54mm:PinHeader_1x04_P2.54mm_Vertical
- U3: footprint Connector_PinHeader_2.54mm:PinHeader_1x04_P2.54mm_Vertical -> Connector_PinHeader_2.54mm:PinHeader_1x04_P2.54mm_Horizontal
Connections:
- net +5V: now also J2.15 (Pin_15)
- net CNY 1: now also J2.13 (Pin_13)
- net CNY 2: now also J2.11 (Pin_11)
- net ECHO 1: now also J2.1 (Pin_1)
- net ECHO 2: now also J2.3 (Pin_3)
- net ECHO 3: now also J2.5 (Pin_5)
- net ECHO 4: now also J2.7 (Pin_7)
- net ECHO 5: now also J2.9 (Pin_9)
- net GND: now also J2.16 (Pin_16)
- net TRIG 1: now also J2.10 (Pin_10)
- net TRIG 2: now also J2.2 (Pin_2)
- net TRIG 3: now also J2.4 (Pin_4)
- net TRIG 4: now also J2.8 (Pin_8)
- net TRIG 5: now also J2.6 (Pin_6)
- no-connect marks 3 -> 4
