File: Electronica/SHAPRS BY DYNER/SHAPRS BY DYNER.kicad_pcb (KiCad board)
At the start: 2 copper layers, 23 x 17.2 mm, 8 parts, among them J1 Conn_01x03_Socket, Q1 2N2222A, Q2 2N2222A

Commit message: .
Parts:
- LED 1: renamed from D1
- LED 2: renamed from D2
Connections:
- J1 pad 3: unconnected-(J1-Pin_3-Pad3) -> pin
Routing:
- net pin: track 0.00 -> 5.37 mm
Changed lines of the file:
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@@
 	(net 4 "Net-(Q1-Pad3)")
 	(net 5 "+5V")
-	(net 6 "unconnected-(J1-Pin_3-Pad3)")
-	(net 7 "Net-(Q1-Pad2)")
-	(net 8 "pin")
+	(net 6 "Net-(Q1-Pad2)")
+	(net 7 "pin")
 	(footprint "LED_THT:LED_D5.0mm"
 		(layer "F.Cu")
@@
 		(descr "LED, diameter 5.0mm, 2 pins, http://cdn-reichelt.de/documents/datenblatt/A500/LL-504BC2E-009.pdf")
 		(tags "LED diameter 5.0mm 2 pins")
-		(property "Reference" "D1"
-			(at 1.27 -3.96 360)
+		(property "Reference" "LED 1"
+			(at -2.86 0.6 90)
 			(layer "F.SilkS")
 			(effects
@@
 		)
 		(property "Value" "LED"
-			(at 1.27 3.96 360)
+			(at 1.27 3.96 0)
 			(layer "F.Fab")
 			(effects
@@
 		)
 		(fp_text user "${REFERENCE}"
-			(at 1.25 0 360)
+			(at 1.25 0 0)
 			(layer "F.Fab")
 			(effects
@@
 		(descr "LED, diameter 5.0mm, 2 pins, http://cdn-reichelt.de/documents/datenblatt/A500/LL-504BC2E-009.pdf")
 		(tags "LED diameter 5.0mm 2 pins")
-		(property "Reference" "D2"
-			(at 1.27 -3.96 360)
+		(property "Reference" "LED 2"
+			(at 5.39 0.6 90)
 			(layer "F.SilkS")
 			(effects
@@
 		)
 		(property "Value" "LED"
-			(at 1.27 3.96 360)
+			(at 1.27 3.96 0)
 			(layer "F.Fab")
 			(effects
@@
 		)
 		(fp_text user "${REFERENCE}"
-			(at 1.25 0 360)
+			(at 1.25 0 0)
 			(layer "F.Fab")
 			(effects
@@
 		)
 		(fp_text user "${REFERENCE}"
-			(at 0 2.54 360)
+			(at 0 2.54 0)
 			(layer "F.Fab")
 			(effects
@@
 			(layers "*.Cu" "*.Mask")
 			(remove_unused_layers no)
-			(net 6 "unconnected-(J1-Pin_3-Pad3)")
+			(net 7 "pin")
 			(pinfunction "Pin_3")
 			(pintype "passive")
@@
 		(at 51.2 28 180)
 		(property "Reference" "Q2"
-			(at 1.04313 -4.08359 360)
+			(at -2.6 4 0)
 			(layer "F.SilkS")
 			(effects
@@
 		)
 		(property "Value" "2N2222A"
-			(at 7.20046 3.72176 360)
+			(at 7.20046 3.72176 0)
 			(layer "F.Fab")
 			(effects
@@
 		)
 		(property "Footprint" "2N2222A:TO127P584H533-3"
-			(at 0 0 360)
+			(at 0 0 0)
 			(layer "F.Fab")
 			(hide yes)
@@
 		)
 		(property "Datasheet" ""
-			(at 0 0 360)
+			(at 0 0 0)
 			(layer "F.Fab")
 			(hide yes)
@@
 		)
 		(property "Description" ""
-			(at 0 0 360)
+			(at 0 0 0)
 			(layer "F.Fab")
 			(hide yes)
@@
 			(layers "*.Cu" "*.Mask")
 			(remove_unused_layers no)
-			(net 8 "pin")
+			(net 7 "pin")
 			(pintype "passive")
 			(solder_mask_margin 0.102)
@@
 			(layers "*.Cu" "*.Mask")
 			(remove_unused_layers no)
-			(net 7 "Net-(Q1-Pad2)")
+			(net 6 "Net-(Q1-Pad2)")
 			(pintype "passive")
 			(solder_mask_margin 0.102)
@@
 		(at 36 27.6)
 		(property "Reference" "Q1"
-			(at 1.04313 -4.08359 360)
+			(at -2 -3.6 0)
 			(layer "F.SilkS")
 			(effects
@@
 		)
 		(property "Value" "2N2222A"
-			(at 3.47 3.4 360)
+			(at 3.47 3.4 0)
 			(layer "F.Fab")
 			(effects
@@
 		)
 		(property "Footprint" "2N2222A:TO127P584H533-3"
-			(at 0 0 360)
+			(at 0 0 0)
 			(layer "F.Fab")
 			(hide yes)
@@
 		)
 		(property "Datasheet" ""
-			(at 0 0 360)
+			(at 0 0 0)
 			(layer "F.Fab")
 			(hide yes)
@@
 		)
 		(property "Description" ""
-			(at 0 0 360)
+			(at 0 0 0)
 			(layer "F.Fab")
 			(hide yes)
@@
 			(layers "*.Cu" "*.Mask")
 			(remove_unused_layers no)
-			(net 7 "Net-(Q1-Pad2)")
+			(net 6 "Net-(Q1-Pad2)")
 			(pintype "passive")
 			(solder_mask_margin 0.102)
@@
 		)
 		(fp_text user "${REFERENCE}"
-			(at 0 0 360)
+			(at 0 0 0)
 			(layer "B.Fab")
 			(effects
@@
 			(layers "B.Cu" "B.Paste" "B.Mask")
 			(roundrect_rratio 0.25)
-			(net 7 "Net-(Q1-Pad2)")
+			(net 6 "Net-(Q1-Pad2)")
 			(pintype "passive")
 		)
@@
 	)
 	(segment
-		(start 45.8 20.127208)
-		(end 46.327208 19.6)
-		(width 0.8)
-		(layer "B.Cu")
-		(net 2)
-	)
-	(segment
 		(start 47.4 32.722352)
 		(end 45.009852 32.722352)
@@
 	)
 	(segment
-		(start 46.327208 19.6)
-		(end 54.5 19.6)
-		(width 0.8)
-		(layer "B.Cu")
-		(net 2)
-	)
-	(segment
-		(start 45.8 21.4)
-		(end 45.8 20.127208)
-		(width 0.8)
-		(layer "B.Cu")
-		(net 2)
-	)
-	(segment
 		(start 51 32.8)
 		(end 54.8 32.8)
@@
 	)
 	(segment
+		(start 45.8 21.4)
+		(end 45.8 19.6)
+		(width 0.8)
+		(layer "B.Cu")
+		(net 2)
+	)
+	(segment
+		(start 45.8 19.6)
+		(end 54.5 19.6)
+		(width 0.8)
+		(layer "B.Cu")
+		(net 2)
+	)
+	(segment
 		(start 39.25 21.4)
 		(end 34 21.4)
@@
 		(width 0.8)
 		(layer "B.Cu")
-		(net 7)
+		(net 6)
 	)
 	(segment
@@
 		(width 0.8)
 		(layer "B.Cu")
-		(net 7)
+		(net 6)
 	)
 	(segment
@@
 		(width 0.8)
 		(layer "B.Cu")
-		(net 7)
+		(net 6)
 	)
 	(segment
@@
 		(width 0.8)
 		(layer "B.Cu")
-		(net 7)
+		(net 6)
 	)
 	(segment
@@
 		(width 0.8)
 		(layer "B.Cu")
-		(net 7)
+		(net 6)
 	)
 	(segment
@@
 		(width 0.8)
 		(layer "B.Cu")
-		(net 7)
+		(net 6)
 	)
 	(segment
@@
 		(width 0.8)
 		(layer "B.Cu")
-		(net 7)
+		(net 6)
 	)
 	(segment
@@
 		(width 0.8)
 		(layer "B.Cu")
+		(net 6)
+	)
+	(segment
+		(start 46.08 26.6)
+		(end 46.68 26)
+		(width 0.8)
+		(layer "B.Cu")
+		(net 7)
+	)
+	(segment
+		(start 46.68 26)
+		(end 51.2 26)
+		(width 0.8)
+		(layer "B.Cu")
