File: Electronica/SHAPRS BY DYNER/SHAPRS BY DYNER.kicad_sch (KiCad schematic)
At the start: 8 parts, among them J1 Conn_01x03_Socket, Q1 2N2222A, Q2 2N2222A

Commit message: .
Connections:
- net pin: now also J1.3 (Pin_3)
Changed lines of the file:
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@@
+	(global_label "pin"
+		(shape input)
+		(at 26.67 46.99 0)
+		(fields_autoplaced yes)
+		(effects
+			(font
+				(size 1.27 1.27)
+			)
+			(justify left)
+		)
+		(property "Intersheetrefs" "${INTERSHEET_REFS}"
+			(at 32.558 46.99 0)
+			(effects
+				(font
+					(size 1.27 1.27)
+				)
+				(justify left)
+				(hide yes)
+			)
+		)
+	)
 	(global_label "pin"
 		(shape input)
