File: Electronica/CNY PLACA DYNER/CNY PLACA DYNER.kicad_sch (KiCad schematic)
At the start: 4 parts, among them J1 Conn_01x03_Socket, U1 CNY70

Commit message: ups
Parts:
- R2: value 10k -> 47K
Changed lines of the file:
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@@
 			)
 		)
-		(property "Value" "10k"
+		(property "Value" "47K"
 			(at 38.862 31.496 90)
 			(effects
