File: Electronica/PCB/PCB Principal V5/PCB Principal V5.kicad_pcb (KiCad board)
At the start: 2 copper layers, 110 x 81.5 mm, 17 parts, among them J12 TP, J2 Power Monster, J4 Power Input 2, J5 IDC Placa Botones, J6 Power Input 1

Commit message: ,
Parts:
- removed Arduino Nano: Arduino_Nano_v3.x, Module:Arduino_Nano
- removed J12: TP, Connector_PinHeader_2.54mm:PinHeader_1x05_P2.54mm_Vertical
- removed Monster Shield: MONSTER SHIELD, Module:Arduino_UNO_R3
- removed Pines Sensores: Conexion Sensores, Connector_PinHeader_2.54mm:PinHeader_2x08_P2.54mm_Horizontal
- removed SW Motores: On/Off Motores, Button_Switch_THT:SW_Slide_SPDT_Angled_CK_OS102011MA1Q
- removed SW On/Off: On/Off General, TerminalBlock:TerminalBlock_bornier-2_P5.08mm
- added A1: Arduino_Nano_v3.x, Module:Arduino_Nano, F.Cu at (222.0, 58.6)
- added A2: MONSTER SHIELD, Module:Arduino_UNO_R3, B.Cu at (275.3, 59.5)
- added J1: Conexion Sensores, Connector_PinHeader_2.54mm:PinHeader_2x08_P2.54mm_Horizontal, F.Cu at (221.5, 73.8)
- added J3: On/Off General, TerminalBlock:TerminalBlock_bornier-2_P5.08mm, F.Cu at (158.5, 58.4)
- added SW1: On/Off Motores, Button_Switch_THT:SW_Slide_SPDT_Angled_CK_OS102011MA1Q, F.Cu at (156.9, 80.1)
- LM1: footprint LM2596:LM2596_correctedMeas -> Step Down:LM2596_correctedMeas
- moved R1 139.1 mm to (165.5, 58.3), turned to -90 degrees
- moved D3 130.5 mm to (160.0, 65.4), turned to -90 degrees
- moved J6 126.1 mm to (158.6, 23.8), turned to -90 degrees
- moved J4 120.6 mm to (170.6, 31.6), turned to 90 degrees
- moved D1 104.3 mm to (168.7, 49.0), turned to 90 degrees
- moved LM1 103.3 mm to (184.2, 58.6)
- moved D2 98.7 mm to (163.9, 49.0), turned to 90 degrees
- moved J5 88.9 mm to (187.8, 31.4)
- moved J2 48.6 mm to (185.4, 84.8), turned to 180 degrees
- moved D4 24.4 mm to (168.5, 77.2)
- moved R2 19.4 mm to (163.4, 73.1), turned to 0 degrees
Connections:
- LM1 pad 4: VIN -> VNano
Routing:
- net GND: track 0.00 -> 427.1 mm
- net +5V: track 0.00 -> 134.1 mm, vias 0 -> 2
- net TRIG 3: track 0.00 -> 70.0 mm
- net LED2: track 0.00 -> 64.5 mm
- net MOTORES: track 0.00 -> 61.9 mm
- net VNano: track 0.00 -> 54.1 mm, vias 0 -> 2
- net LED3: track 0.00 -> 53.5 mm
- net ECHO 1: track 0.00 -> 52.2 mm
- net TRIG 1: track 0.00 -> 48.7 mm
- net ECHO 2: track 0.00 -> 45.3 mm
- net TRIG 2: track 0.00 -> 42.4 mm
- net Net-(J2-Pin_2): track 0.00 -> 39.7 mm
- net CNY 1: track 0.00 -> 34.3 mm
- net CNY 2: track 0.00 -> 30.2 mm
- net Net-(D3-A): track 0.00 -> 19.7 mm
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Other:
- board size 110 x 81.5 mm -> 130.5 x 70 mm

Commit message: .
Parts:
- moved LM1 21.7 mm to (163.6, 65.6)
- moved A1 21.7 mm to (201.5, 65.5)
- moved D2 21.7 mm to (143.4, 55.9)
- moved D4 21.7 mm to (148.0, 84.2)
- moved J2 21.7 mm to (164.9, 91.8)
- moved J3 21.7 mm to (138.0, 65.4)
- moved R1 21.7 mm to (145.0, 65.2)
- moved SW1 21.7 mm to (136.4, 87.0)
- moved A2 21.7 mm to (254.7, 66.5)
- moved D1 21.7 mm to (148.2, 55.9)
- moved D3 21.7 mm to (139.4, 72.4)
- moved J1 21.7 mm to (200.9, 80.7)
- moved J4 21.7 mm to (150.1, 38.6)
- moved J5 21.7 mm to (167.3, 38.3)
- moved J6 21.7 mm to (138.1, 30.8)
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Routing:
- net ECHO 3: track 0.00 -> 79.0 mm, vias 0 -> 2
- net GND: track 427.1 -> 439.8 mm
- net Net-(D1-K): track 14.6 -> 12.1 mm
- net MOTORES: track 61.9 -> 64.3 mm
- net Net-(J2-Pin_2): track 39.7 -> 40.8 mm
- net (no net): vias 0 -> 2
Other:
- board size 130.5 x 70 mm -> 139.1 x 70 mm
- board text added: "Chiken Litlle"

Commit message: -
Parts:
- added J12: TP, Connector_PinHeader_2.54mm:PinHeader_1x05_P2.54mm_Vertical, F.Cu at (129.3, 43.7)
Routing:
- net VNano: track 54.1 -> 81.0 mm
- net GND: track 439.8 -> 458.1 mm
- net PI+: track 17.9 -> 26.7 mm
- net +5V: track 134.1 -> 129.8 mm

Commit message: ok
Parts:
- added J7: Conn_01x01_Pin, Connector_PinHeader_2.54mm:PinHeader_1x01_P2.54mm_Vertical, F.Cu at (138.8, 52.5)
- added J8: Conn_01x01_Pin, Connector_PinHeader_2.54mm:PinHeader_1x01_P2.54mm_Vertical, F.Cu at (134.3, 53.7)
- moved D3 38.7 mm to (173.8, 90.2)
- moved J2 34.1 mm to (136.2, 73.3), turned to -90 degrees
- moved R1 28.2 mm to (154.3, 91.8), turned to 0 degrees
Routing:
- net GND: track 458.1 -> 401.3 mm
- net Net-(J2-Pin_2): track 40.8 -> 16.4 mm
- net Net-(D3-A): track 19.8 -> 12.2 mm
- net +5V: track 129.8 -> 136.3 mm
- net ECHO 3: track 79.0 -> 83.5 mm
- net BTN2: track 19.3 -> 18.7 mm

Commit message: .
Parts:
- removed J7, J8: Conn_01x01_Pin, Connector_PinHeader_2.54mm:PinHeader_1x01_P2.54mm_Vertical
- added ?: , , F.Cu at (261.9, 91.2)
- added ?: , , F.Cu at (129.8, 31.0)
- moved D3 7.25 mm to (166.6, 91.3), turned to 0 degrees
Routing:
- net GND: track 401.3 -> 453.3 mm
- net +5V: track 136.3 -> 126.3 mm
- net (no net): vias 2 -> 0

Commit message: PCB V5 LINDA HERMOSA DIVINA
Parts:
- removed the ? at (261.9, 91.2)
- removed the ? at (129.8, 31.0)
- removed J12: TP, Connector_PinHeader_2.54mm:PinHeader_1x05_P2.54mm_Vertical
- removed J5: IDC Placa Botones, Connector_PinHeader_2.54mm:PinHeader_2x05_P2.54mm_Horizontal
- added ?: , , F.Cu at (109.0, 47.0)
- added ?: , , F.Cu at (230.0, 118.6)
- added J11: Conn_01x04_Pin, Connector_PinHeader_2.54mm:PinHeader_1x04_P2.54mm_Vertical, F.Cu at (153.5, 47.6)
- added J7: Placa de Botones, Connector_PinHeader_2.54mm:PinHeader_2x04_P2.54mm_Horizontal, F.Cu at (210.8, 58.2)
- added U1: 74HC595, 74HC595N_DIP16_:DIP16-2.54-20.32X5.84MM, B.Cu at (201.4, 68.6)
- J1: moved to B.Cu
- LM1: footprint Step Down:LM2596_correctedMeas -> StepDown:StepDown
- SW1: footprint Button_Switch_THT:SW_Slide_SPDT_Angled_CK_OS102011MA1Q -> Button_Switch_THT:SW_Slide_SPDT_Straight_CK_OS102011MS2Q
- moved A2 117.4 mm to (137.9, 78.0), turned to -90 degrees
- moved J3 55.2 mm to (114.1, 115.2), turned to 180 degrees
- moved LM1 46.2 mm to (123.0, 87.4)
- moved J2 45.0 mm to (119.9, 115.2), turned to 0 degrees
- moved J4 32.5 mm to (119.9, 50.4), turned to 0 degrees
- moved D1 30.1 mm to (118.1, 57.4), turned to 0 degrees
- moved J1 28.4 mm to (187.5, 55.7)
- moved SW1 27.3 mm to (131.9, 114.0), turned to -90 degrees
- moved R2 27.3 mm to (148.8, 106.7)
- moved D4 27.0 mm to (153.9, 110.5)
- moved D2 26.1 mm to (118.1, 62.4), turned to 0 degrees
- moved J6 19.7 mm to (139.2, 50.4), turned to 0 degrees
- moved D3 19.6 mm to (170.3, 110.5)
- moved R1 18.5 mm to (165.3, 106.7)
- moved A1 13.2 mm to (199.4, 78.5), turned to 0 degrees
Connections:
- A1 pad 11: TRIG 2 -> ECHO 1
- A1 pad 13: TRIG 1 -> ECHO 3
- A1 pad 14: ECHO 1 -> Data
- A1 pad 15: ECHO 3 -> Latch
- A1 pad 16: LED4 -> Clock
- A1 pad 19: LED1 -> unconnected-(A1-A0-Pad19)
- A1 pad 20: BTN1 -> ECHO 4
- A1 pad 21: BTN2 -> ECHO 5
- A1 pad 22: TRIG 3 -> LED1
- A1 pad 23: LED3 -> BTN1
- A1 pad 24: LED2 -> BTN2
- A1 pad 25: CNY 1 -> CNY 2
- A1 pad 26: CNY 2 -> CNY 1
- J1 pad 1: TRIG 2 -> ECHO 1
- J1 pad 10: TRIG 4 -> TRIG 1
- J1 pad 12: ECHO 5 -> unconnected-(J1-Pin_12-Pad12)
- J1 pad 13: CNY 3 -> CNY 1
- J1 pad 14: TRIG 5 -> unconnected-(J1-Pin_14-Pad14)
- J1 pad 2: ECHO 3 -> TRIG 2
- J1 pad 5: TRIG 1 -> ECHO 3
- J1 pad 6: unconnected-(J1-Pin_6-Pad6) -> TRIG 5
- J1 pad 7: ECHO 1 -> ECHO 4
- J1 pad 8: ECHO 4 -> TRIG 4
- J1 pad 9: CNY 1 -> ECHO 5
Routing:
- net VNano: track 81.0 -> 244.9 mm
- net ECHO 4: track 0.00 -> 123.6 mm
- net ECHO 5: track 0.00 -> 111.6 mm
- net +5V: track 126.3 -> 228.7 mm, vias 2 -> 4
- net ECHO 2: track 45.3 -> 116.2 mm
- net GND: track 453.3 -> 385.7 mm, vias 0 -> 8
- net CNY 2: track 30.2 -> 92.0 mm, vias 0 -> 2
- net TRIG 3: track 70.0 -> 8.61 mm
- net LED2: track 64.5 -> 12.2 mm
- net Latch: track 0.00 -> 50.7 mm
- net Data: track 0.00 -> 50.1 mm
- net Net-(D1-K): track 12.1 -> 61.7 mm
- net Clock: track 0.00 -> 49.2 mm
- net CNY 1: track 34.3 -> 80.4 mm, vias 0 -> 2
- net ECHO 3: track 83.5 -> 127.0 mm, vias 2 -> 0
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Other:
- board size 139.1 x 70 mm -> 127.5 x 78.4 mm
- board text added: "(¬_¬ )"
- board text added: "(⊙_⊙;)"
- board text added: "CDR 2024"
- board text added: "Chicken Little V5"
- board text added: "^_^"
- board text removed: "Chiken Litlle"

Commit message: PCB Principal V5 terminada
Parts:
- moved SW1 0.80 mm to (132.7, 114.0)
- moved U1 0.40 mm to (201.4, 68.2)
Connections:
- A1 pad 27: +5V -> unconnected-(A1-+5V-Pad27)
- A1 pad 30: VNano -> +5V
- A2 pad 8: VIN -> +5V
- D1 pad 2: PI+ -> Net-(D1-A)
- D2 pad 2: PI+ -> Net-(D1-A)
- J11 pad 1: PI+ -> +24V
- J11 pad 2: VNano -> +5V
- J11 pad 3: +5V -> unconnected-(J11-Pin_3-Pad3)
- J3 pad 1: MOTORES -> +24V
- J6 pad 2: PI+ -> Net-(D1-A)
- LM1 pad 2: MOTORES -> +24V
- LM1 pad 4: VNano -> +5V
- R1 pad 1: MOTORES -> +24V
- SW1 pad 2: MOTORES -> +24V
Routing:
- net VNano: track 244.9 -> 0.00 mm, vias 2 -> 0
- net +5V: track 228.7 -> 463.5 mm, vias 4 -> 6
- net +24V: track 0.00 -> 158.8 mm, vias 0 -> 2
- net MOTORES: track 78.0 -> 0.00 mm
- net PI+: track 38.4 -> 0.00 mm
- net Net-(D1-A): track 0.00 -> 29.4 mm
- net BTN1: track 46.0 -> 49.0 mm
- net BTN2: track 42.3 -> 45.1 mm
- net LED1: track 50.1 -> 52.9 mm
- net LED4: track 37.2 -> 35.4 mm
- net CNY 1: track 80.4 -> 79.3 mm
- net LED3: track 58.2 -> 57.2 mm
- net ECHO 4: track 123.6 -> 122.9 mm
- net ECHO 5: track 111.6 -> 110.8 mm
- net CNY 2: track 92.0 -> 91.4 mm
