File: Electronica/PCB/PCB Principal V5/PCB Principal V5.kicad_pcb (KiCad board)
At the start: 2 copper layers, 127.5 x 78.4 mm, 20 parts, among them J1 Conexion Sensores, J11 Conn_01x04_Pin, J2 Power Monster, J3 On/Off General, J4 Power Input 2, J6 Power Input 1, J7 Placa de Botones, SW1 On/Off Motores, U1 74HC595

Commit message: seligrafiaskfbvlajBSJFV
TONTO EL Q LEE
Parts:
- LM 2596: renamed from LM1
- PLACA : renamed from J1
- moved SW1 1.29 mm to (131.4, 114.1)
- renumbered U1 to 74HC595, J7 to BOTONES, A1 to NANO, J11 to TP
Routing:
- net +24V: track 158.8 -> 160.4 mm
- net Net-(J2-Pin_2): track 36.4 -> 37.9 mm
Other:
- board text added: "24V"
- board text added: "5V"
- board text added: "GND"
- board text added: "I"
- board text added: "MONSTER SHIELD"
- board text added: "PLACA"
- board text added: "SENSORES"
