File: Electronica/PCB/PCB de botones V2/PCB de botones V2.kicad_sch (KiCad schematic)
At the start: 11 parts, among them J1 IDC Placa Botones, SW1 SW_Push, SW2 SW_Push

Commit message: prueba de botones, contador binario
Changed lines of the file:
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@@
-		)
-	)
-	(symbol
-		(lib_id "power:+5V")
-		(at 71.12 15.24 90)
-		(unit 1)
-		(exclude_from_sim no)
-		(in_bom yes)
-		(on_board yes)
-		(dnp no)
-		(fields_autoplaced yes)
-		(property "Reference" "#PWR04"
-			(at 74.93 15.24 0)
-			(effects
-				(font
-					(size 1.27 1.27)
-				)
-				(hide yes)
-			)
-		)
-		(property "Value" "+5V"
-			(at 67.31 15.2399 90)
-			(effects
-				(font
-					(size 1.27 1.27)
-				)
-				(justify left)
-			)
-		)
-		(property "Footprint" ""
-			(at 71.12 15.24 0)
-			(effects
-				(font
-					(size 1.27 1.27)
-				)
-				(hide yes)
-			)
-		)
-		(property "Datasheet" ""
-			(at 71.12 15.24 0)
-			(effects
-				(font
-					(size 1.27 1.27)
-				)
-				(hide yes)
-			)
-		)
-		(property "Description" "Power symbol creates a global label with name \"+5V\""
-			(at 71.12 15.24 0)
-			(effects
-				(font
-					(size 1.27 1.27)
-				)
-				(hide yes)
-			)
-		)
-		(pin "1"
-		)
-		(instances
-			(project "PCB de botones V2"
-				(path "/83e621f7-046b-4df3-a825-7f5b54a0265f"
-					(reference "#PWR04")
-					(unit 1)
-				)
-			)
 		)
 	)
