File: Electronica/PCB/PCB Principal V7 - V2/PCB Principal V7.kicad_pcb (KiCad board)
At the start: 2 copper layers, 121 x 65.4 mm, 17 parts

Commit message: V7-V2 TERMINADISIMA
Other:
- board text added: "CHICKEN LITTLE"
- board text added: "DIJO"
- board text added: "SE CAE EL CIELO"
Changed lines of the file:
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@@
 		(layer "Edge.Cuts")
+	)
+	(gr_text "CHICKEN LITTLE"
+		(at 129.824094 70.475 0)
+		(layer "F.SilkS")
+		(effects
+			(font
+				(size 2 2)
+				(thickness 0.4)
+				(bold yes)
+			)
+			(justify left bottom)
+		)
 	)
 	(gr_text "Step Down"
@@
 				(size 1 1)
 				(thickness 0.15)
+			)
+			(justify left bottom)
+		)
+	)
+	(gr_text "DIJO"
+		(at 139.221714 65.9 0)
+		(layer "F.SilkS")
+		(effects
+			(font
+				(size 1.5 1.5)
+				(thickness 0.3)
+				(bold yes)
 			)
 			(justify left bottom)
@@
 			)
 			(justify left bottom)
+		)
+	)
+	(gr_text "SE CAE EL CIELO "
+		(at 131.471714 62.65 0)
+		(layer "F.SilkS")
+		(effects
+			(font
+				(size 1.5 1.5)
+				(thickness 0.3)
+				(bold yes)
+			)
+			(justify left bottom)

Commit message: .
Parts:
- J1: renamed from Placa de Sensores
- J2: renamed from Power Monster 
- SW2: renamed from Dip Switch
- renumbered Nano to A1, On/Off to D3, Motores to D4, 24V to J3, XT60 to J6, LM2596 to LM1, On/Off to SW1, Start to SW3, 74hc4067 to U2
Changed lines of the file:
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@@
 		)
 		(property ki_fp_filters "D*DO?41*")
-		(sheetname "Root")
+		(sheetname "Raíz")
 		(sheetfile "PCB Principal V7.kicad_sch")
 		(attr through_hole)
@@
 		(descr "Arduino Nano, http://www.mouser.com/pdfdocs/Gravitech_Arduino_Nano3_0.pdf")
 		(tags "Arduino Nano")
-		(property "Reference" "Nano"
+		(property "Reference" "A1"
 			(at 0.154 -5.08 0)
 			(layer "F.SilkS")
@@
 		)
 		(property ki_fp_filters "Arduino*Nano*")
-		(sheetname "Root")
+		(sheetname "Raíz")
 		(sheetfile "PCB Principal V7.kicad_sch")
 		(attr through_hole)
@@
 		(descr "simple 2-pin terminal block, pitch 5.08mm, revamped version of bornier2")
 		(tags "terminal block bornier2")
-		(property "Reference" "Power Monster "
+		(property "Reference" "J2"
 			(at 2.29 5.093 0)
 			(layer "F.SilkS")
@@
 		)
 		(property ki_fp_filters "TerminalBlock*:*")
-		(sheetname "Root")
+		(sheetname "Raíz")
 		(sheetfile "PCB Principal V7.kicad_sch")
 		(attr through_hole)
@@
 		)
 		(property ki_fp_filters "R_*")
-		(sheetname "Root")
+		(sheetname "Raíz")
 		(sheetfile "PCB Principal V7.kicad_sch")
 		(attr through_hole)
@@
 		(descr "LED, diameter 5.0mm z-position of LED center 3.0mm, 2 pins")
 		(tags "LED diameter 5.0mm z-position of LED center 3.0mm 2 pins")
-		(property "Reference" "Motores"
+		(property "Reference" "D4"
 			(at -5.147 5.597 0)
 			(layer "F.SilkS")
@@
 		)
 		(property ki_fp_filters "LED* LED_SMD:* LED_THT:*")
-		(sheetname "Root")
+		(sheetname "Raíz")
 		(sheetfile "PCB Principal V7.kicad_sch")
 		(attr through_hole)
@@
 		(descr "CuK miniature slide switch, OS series, SPDT, right angle, http://www.ckswitches.com/media/1428/os.pdf")
 		(tags "switch SPDT")
-		(property "Reference" "On/Off"
+		(property "Reference" "SW1"
 			(at 5.261 3.774 0)
 			(layer "F.SilkS")
@@
 			)
 		)
-		(sheetname "Root")
+		(sheetname "Raíz")
 		(sheetfile "PCB Principal V7.kicad_sch")
 		(attr through_hole)
@@
 		)
 		(property ki_fp_filters "D*DO?41*")
-		(sheetname "Root")
+		(sheetname "Raíz")
 		(sheetfile "PCB Principal V7.kicad_sch")
 		(attr through_hole)
@@
 		(descr "simple 2-pin terminal block, pitch 5.08mm, revamped version of bornier2")
 		(tags "terminal block bornier2")
-		(property "Reference" "24V"
+		(property "Reference" "J3"
 			(at 6.501 -4.901 0)
 			(layer "F.SilkS")
@@
 			)
 		)
-		(sheetname "Root")
+		(sheetname "Raíz")
 		(sheetfile "PCB Principal V7.kicad_sch")
 		(attr through_hole)
@@
 		(descr "5x-dip-switch SPST , Slide, row spacing 7.62 mm (300 mils), body size 9.78x14.88mm (see e.g. https://www.ctscorp.com/wp-content/uploads/206-208.pdf)")
 		(tags "DIP Switch SPST Slide 7.62mm 300mil")
-		(property "Reference" "Dip Switch"
+		(property "Reference" "SW2"
 			(at -2.1325 5.2 180)
 			(layer "F.SilkS")
@@
 		)
 		(property ki_fp_filters "SW?DIP?x5*")
-		(sheetname "Root")
+		(sheetname "Raíz")
 		(sheetfile "PCB Principal V7.kicad_sch")
 		(attr through_hole)
@@
 		(descr "AMASS female XT60, through hole, vertical, https://www.tme.eu/Document/2d152ced3b7a446066e6c419d84bb460/XT60%20SPEC.pdf")
 		(tags "XT60 female vertical")
-		(property "Reference" "XT60"
+		(property "Reference" "J6"
 			(at -1.215 -5.472 180)
 			(layer "F.SilkS")
@@
 		)
 		(property ki_fp_filters "TerminalBlock*:*")
-		(sheetname "Root")
+		(sheetname "Raíz")
 		(sheetfile "PCB Principal V7.kicad_sch")
 		(attr through_hole)
@@
 		(descr "LED, diameter 5.0mm z-position of LED center 3.0mm, 2 pins")
 		(tags "LED diameter 5.0mm z-position of LED center 3.0mm 2 pins")
-		(property "Reference" "On/Off"
+		(property "Reference" "D3"
 			(at 7.349 6.377 0)
 			(layer "F.SilkS")
@@
 		)
 		(property ki_fp_filters "LED* LED_SMD:* LED_THT:*")
-		(sheetname "Root")
+		(sheetname "Raíz")
 		(sheetfile "PCB Principal V7.kicad_sch")
 		(attr through_hole)
@@
 		(descr "Generic 6mm SW tactile push button")
 		(tags "tact sw push 6mm")
-		(property "Reference" "Start"
+		(property "Reference" "SW3"
 			(at -3.95 5.15 0)
 			(layer "F.SilkS")
@@
 		)
 		(property "Value" "SW_Push"
-			(at 3.75 6.7 360)
+			(at 3.75 6.7 0)
 			(layer "F.Fab")
 			(effects
@@
 			)
 		)
-		(sheetname "Root")
+		(sheetname "Raíz")
 		(sheetfile "PCB Principal V7.kicad_sch")
 		(attr through_hole)
@@
 		)
 		(fp_text user "${REFERENCE}"
-			(at 3.25 2.25 360)
+			(at 3.25 2.25 0)
 			(layer "F.Fab")
 			(effects
@@
 		(descr "Through hole angled pin header, 2x08, 2.54mm pitch, 6mm pin length, double rows")
 		(tags "Through hole angled pin header THT 2x08 2.54mm double row")
-		(property "Reference" "Placa de Sensores"
+		(property "Reference" "J1"
 			(at -2.6 8.675 180)
 			(layer "F.SilkS")
@@
 		)
 		(property ki_fp_filters "Connector*:*_2x??_*")
-		(sheetname "Root")
+		(sheetname "Raíz")
 		(sheetfile "PCB Principal V7.kicad_sch")
 		(attr through_hole)
@@
 		(layer "F.Cu")
 		(at 99.314 87.376 180)
-		(property "Reference" "LM2596"
+		(property "Reference" "LM1"
 			(at 0 2.5 0)
 			(layer "F.SilkS")
@@
 			)
 		)
-		(sheetname "Root")
+		(sheetname "Raíz")
 		(sheetfile "PCB Principal V7.kicad_sch")
 		(attr through_hole)
@@
 		)
 		(property ki_fp_filters "R_*")
-		(sheetname "Root")
+		(sheetname "Raíz")
 		(sheetfile "PCB Principal V7.kicad_sch")
 		(attr through_hole)
@@
 		)
 		(property ki_fp_filters "Arduino*UNO*R3*")
-		(sheetname "Root")
+		(sheetname "Raíz")
 		(sheetfile "PCB Principal V7.kicad_sch")
 		(attr through_hole)
@@
 		(descr "SOIC, 24 Pin (JEDEC MS-013AD, https://www.analog.com/media/en/package-pcb-resources/package/pkg_pdf/soic_wide-rw/RW_24.pdf), generated with kicad-footprint-generator ipc_gullwing_generator.py")
 		(tags "SOIC SO")
-		(property "Reference" "74hc4067"
+		(property "Reference" "U2"
 			(at 7.25 0.285 0)
 			(layer "F.SilkS")
@@
 		)
 		(property "Value" "CD74HC4067M"
-			(at 0 -8.65 270)
+			(at 0 -8.65 -90)
 			(layer "B.Fab")
 			(effects
@@
 		)
 		(property ki_fp_filters "SOIC*W*7.5x15.4mm*P1.27mm*")
-		(sheetname "Root")
+		(sheetname "Raíz")
 		(sheetfile "PCB Principal V7.kicad_sch")
 		(attr smd)
@@
 		)
 		(fp_text user "${REFERENCE}"
-			(at 0 0 270)
+			(at 0 0 -90)
 			(layer "B.Fab")
 			(effects
@@
 	)
 	(gr_text "74HC4067"
-		(at 192.9 79.375 0)
+		(at 210.312 82.042 0)
 		(layer "F.SilkS")
 		(effects
@@
 	)
 	(segment
-		(start 200.625 78.711782)
-		(end 201.26 79.346782)
+		(start 200.625 76.704634)
+		(end 201.26 77.339634)
 		(width 0.7)
 		(layer "B.Cu")
@@
 	)
 	(segment
-		(start 200.625 59.45)
-		(end 200.625 78.711782)
+		(start 188.56 59.335)
+		(end 200.51 59.335)
 		(width 0.7)
 		(layer "B.Cu")
@@
 	)
 	(segment
-		(start 188.56 59.335)
-		(end 200.51 59.335)
+		(start 188.56 60.935)
+		(end 188.56 59.335)
 		(width 0.7)
 		(layer "B.Cu")
@@
 	)
 	(segment
-		(start 200.51 59.335)
-		(end 200.625 59.45)
+		(start 201.26 77.339634)
+		(end 201.26 80.95)
 		(width 0.7)
 		(layer "B.Cu")
@@
 	)
 	(segment
-		(start 188.56 60.935)
-		(end 188.56 59.335)
+		(start 200.625 59.45)
+		(end 200.625 76.704634)
 		(width 0.7)
 		(layer "B.Cu")
@@
 	)
 	(segment
-		(start 201.26 79.346782)
-		(end 201.26 80.95)
+		(start 200.51 59.335)
+		(end 200.625 59.45)
 		(width 0.7)
 		(layer "B.Cu")
@@
 	)
 	(segment
-		(start 191.1 78.1)
-		(end 191.1 63.475)
-		(width 0.7)
-		(layer "B.Cu")
-		(net 40)
-	)
-	(segment
-		(start 198.15 79.348052)
-		(end 198.15 78.1)
+		(start 198.72 80.95)
+		(end 198.72 78.959)
 		(width 0.7)
 		(layer "B.Cu")
@@
 	)
 	(segment
-		(start 198.72 80.95)
-		(end 198.72 79.918052)
+		(start 198.72 78.959)
+		(end 197.861 78.1)
 		(width 0.7)
 		(layer "B.Cu")
@@
 	)
 	(segment
-		(start 198.15 78.1)
+		(start 197.861 78.1)
 		(end 191.1 78.1)
 		(width 0.7)
@@
 	)
 	(segment
-		(start 198.72 79.918052)
-		(end 198.15 79.348052)
+		(start 191.1 78.1)
+		(end 191.1 63.475)
 		(width 0.7)
 		(layer "B.Cu")
@@
 	)
 	(segment
-		(start 199.99 79.632417)
-		(end 199.99 80.95)
+		(start 198.595 76.675)
+		(end 199.99 78.07)
 		(width 0.7)
 		(layer "B.Cu")
@@
 	(segment
 		(start 193.64 76.675)
-		(end 199.35 76.675)
-		(width 0.7)
-		(layer "B.Cu")
-		(net 42)
-	)
-	(segment
-		(start 193.64 63.475)
-		(end 193.64 76.675)
+		(end 198.595 76.675)
 		(width 0.7)
 		(layer "B.Cu")
@@
 	)
 	(segment
-		(start 199.35 76.675)
-		(end 199.35 78.992417)
+		(start 199.99 78.07)
+		(end 199.99 80.95)
 		(width 0.7)
 		(layer "B.Cu")
@@
 	)
 	(segment
-		(start 199.35 78.992417)
-		(end 199.99 79.632417)
+		(start 193.64 63.475)
+		(end 193.64 76.675)
 		(width 0.7)
 		(layer "B.Cu")
@@
 	)
 	(segment
-		(start 201.8 58.55)
-		(end 201.425 58.175)
+		(start 202.53 76.292)
+		(end 201.8 75.562)
 		(width 0.7)
 		(layer "B.Cu")
@@
 	)
 	(segment
-		(start 186.02 58.175)
-		(end 186.02 60.935)
+		(start 201.8 75.562)
+		(end 201.8 58.55)
 		(width 0.7)
 		(layer "B.Cu")
@@
 	)
 	(segment
-		(start 201.8 78.331147)
-		(end 201.8 58.55)
+		(start 201.8 58.55)
+		(end 201.425 58.175)
 		(width 0.7)
 		(layer "B.Cu")
@@
 	)
 	(segment
-		(start 201.425 58.175)
-		(end 186.02 58.175)
+		(start 202.53 80.95)
+		(end 202.53 76.292)
 		(width 0.7)
 		(layer "B.Cu")
@@
 	)
 	(segment
-		(start 202.53 80.95)
-		(end 202.53 79.061147)
+		(start 186.02 58.175)
+		(end 186.02 60.935)
 		(width 0.7)
 		(layer "B.Cu")
@@
 	)
 	(segment
-		(start 202.53 79.061147)
-		(end 201.8 78.331147)
+		(start 201.425 58.175)
+		(end 186.02 58.175)
 		(width 0.7)
 		(layer "B.Cu")

Commit message: Sensores V3
Parts:
- R1 910: renamed from R1
- R2 1K: renamed from R2
Routing:
- net +5V: track 259.5 -> 267.3 mm, vias 4 -> 6
- net +24V: track 145.8 -> 145.9 mm, vias 2 -> 0
- net GND: vias 4 -> 6
Changed lines of the file:
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@@
 		(descr "Resistor, Axial_DIN0204 series, Axial, Horizontal, pin pitch=7.62mm, 0.167W, length*diameter=3.6*1.6mm^2, http://cdn-reichelt.de/documents/datenblatt/B400/1_4W%23YAG.pdf")
 		(tags "Resistor Axial_DIN0204 series Axial Horizontal pin pitch 7.62mm 0.167W length 3.6mm diameter 1.6mm")
-		(property "Reference" "R1"
+		(property "Reference" "R1 910"
 			(at 3.81 -1.92 90)
 			(layer "F.SilkS")
@@
 		(descr "Resistor, Axial_DIN0204 series, Axial, Horizontal, pin pitch=7.62mm, 0.167W, length*diameter=3.6*1.6mm^2, http://cdn-reichelt.de/documents/datenblatt/B400/1_4W%23YAG.pdf")
 		(tags "Resistor Axial_DIN0204 series Axial Horizontal pin pitch 7.62mm 0.167W length 3.6mm diameter 1.6mm")
-		(property "Reference" "R2"
+		(property "Reference" "R2 1K"
 			(at 3.81 -1.92 0)
 			(layer "F.SilkS")
@@
 	)
 	(gr_line
+		(start 121.425 88.725)
+		(end 121.425 93.8)
+		(stroke
+			(width 1)
+			(type default)
+		)
+		(layer "F.SilkS")
+	)
+	(gr_line
 		(start 189.046875 72.78125)
 		(end 198.875 72.725)
@@
 	)
 	(gr_line
-		(start 112.721875 91.38125)
-		(end 124.3 91.425)
+		(start 112.875 88.85)
+		(end 112.7 94.1)
 		(stroke
 			(width 1)
@@
 	)
 	(segment
+		(start 121.425 88.725)
+		(end 121.425 93.825)
+		(width 1)
+		(layer "F.Cu")
+		(net 10)
+	)
+	(segment
 		(start 198.575 70.175)
 		(end 189.1 70.175)
@@
 	)
 	(via
+		(at 121.425 93.825)
+		(size 1.8)
+		(drill 1)
+		(layers "F.Cu" "B.Cu")
+		(net 10)
+	)
+	(via
 		(at 198.575 70.175)
 		(size 1.8)
@@
 	)
 	(via
+		(at 121.425 88.725)
+		(size 1.8)
+		(drill 1)
+		(layers "F.Cu" "B.Cu")
+		(net 10)
+	)
+	(via
 		(at 189.05 70.125)
 		(size 1.8)
@@
 	)
 	(segment
-		(start 121.37 86.54)
-		(end 121.37 102.18)
-		(width 1)
-		(layer "B.Cu")
-		(net 10)
-	)
-	(segment
 		(start 117.856 86.36)
 		(end 119.78 86.36)
@@
 	)
 	(segment
+		(start 121.425 93.825)
+		(end 121.425 102.125)
+		(width 1)
+		(layer "B.Cu")
+		(net 10)
+	)
+	(segment
 		(start 181.9 70.125)
 		(end 181.775 70.25)
@@
 	)
 	(segment
+		(start 121.425 102.125)
+		(end 121.37 102.18)
+		(width 1)
+		(layer "B.Cu")
+		(net 10)
+	)
+	(segment
 		(start 167.916 69.584)
 		(end 167.916 56.784)
@@
 	)
 	(segment
+		(start 121.37 88.67)
+		(end 121.425 88.725)
+		(width 1)
+		(layer "B.Cu")
+		(net 10)
+	)
+	(segment
 		(start 163.85 107.8)
 		(end 163.85 69.775)
@@
 	)
 	(segment
+		(start 121.37 86.54)
+		(end 121.37 88.67)
+		(width 1)
+		(layer "B.Cu")
+		(net 10)
+	)
+	(segment
 		(start 196.18 60.935)
 		(end 197.76 60.935)
@@
 	)
 	(segment
+		(start 112.725 89.05)
+		(end 112.875 88.9)
+		(width 1)
+		(layer "F.Cu")
+		(net 18)
+	)
+	(segment
+		(start 112.725 94.075)
+		(end 112.725 89.05)
+		(width 1)
+		(layer "F.Cu")
+		(net 18)
+	)
+	(segment
 		(start 189.125 72.725)
 		(end 198.825 72.725)
@@
 	)
 	(via
+		(at 112.875 88.9)
+		(size 1.8)
+		(drill 1)
+		(layers "F.Cu" "B.Cu")
+		(net 18)
+	)
+	(via
 		(at 189.05 72.8)
 		(size 1.8)
@@
 		(net 18)
 	)
+	(via
+		(at 112.725 94.075)
+		(size 1.8)
+		(drill 1)
+		(layers "F.Cu" "B.Cu")
+		(net 18)
+	)
 	(segment
 		(start 196.18 72.75)
@@
 	)
 	(segment
-		(start 117.856 88.9)
-		(end 117.856 93.98)
-		(width 1)
-		(layer "B.Cu")
-		(net 18)
-	)
-	(segment
 		(start 203.725 54.725)
 		(end 203.8 54.8)
@@
 	)
 	(segment
+		(start 117.856 93.98)
+		(end 112.82 93.98)
+		(width 1)
+		(layer "B.Cu")
+		(net 18)
+	)
+	(segment
 		(start 198.775 75.225)
 		(end 198.775 75.575)
@@
 	)
 	(segment
+		(start 112.82 93.98)
+		(end 112.725 94.075)
+		(width 1)
+		(layer "B.Cu")
+		(net 18)
+	)
+	(segment
+		(start 112.875 88.9)
+		(end 115.316 88.9)
+		(width 1)
+		(layer "B.Cu")
+		(net 18)
+	)
+	(segment
 		(start 189.05 72.8)
 		(end 186.436 72.8)
@@
 	)
 	(segment
-		(start 112.7 91.4)
-		(end 124.175 91.4)
-		(width 2)
-		(layer "F.Cu")
-		(net 52)
-	)
-	(segment
-		(start 124.175 91.4)
-		(end 124.225 91.45)
-		(width 2)
-		(layer "F.Cu")
-		(net 52)
-	)
-	(via
-		(at 112.7 91.4)
-		(size 1.8)
-		(drill 1)
-		(layers "F.Cu" "B.Cu")
-		(net 52)
-	)
-	(via
-		(at 124.225 91.45)
-		(size 1.8)
-		(drill 1)
-		(layers "F.Cu" "B.Cu")
-		(net 52)
-	)
-	(segment
 		(start 86.36 91.45)
 		(end 86.36 103.172)
@@
 	)
 	(segment
-		(start 153.421 91.521)
-		(end 153.421 94.737)
-		(width 2)
-		(layer "B.Cu")
-		(net 52)
-	)
-	(segment
 		(start 86.36 52.41)
 		(end 86.36 91.45)
@@
 	)
 	(segment
-		(start 112.7 91.4)
-		(end 86.41 91.4)
-		(width 2)
+		(start 153.421 91.475)
+		(end 86.385 91.475)
+		(width 0.7)
 		(layer "B.Cu")
 		(net 52)
@@
 	)
 	(segment
-		(start 86.41 91.4)
-		(end 86.36 91.45)
-		(width 2)
-		(layer "B.Cu")
-		(net 52)
-	)
-	(segment
 		(start 95.904 107.376)
 		(end 95.904 103.126)
@@
 	)
 	(segment
+		(start 153.421 94.737)
+		(end 153.421 91.475)
+		(width 0.7)
+		(layer "B.Cu")
+		(net 52)
+	)
+	(segment
 		(start 95.904 103.126)
 		(end 95.96 103.07)
@@
 	)
 	(segment
-		(start 153.35 91.45)
-		(end 153.421 91.521)
+		(start 86.41 91.4)
+		(end 86.36 91.45)
 		(width 2)
 		(layer "B.Cu")
@@
 	)
 	(segment
-		(start 124.225 91.45)
-		(end 153.35 91.45)
-		(width 2)
+		(start 86.385 91.475)
+		(end 86.36 91.45)
+		(width 0.7)
 		(layer "B.Cu")
 		(net 52)

Commit message: Placa principal terminada
Parts:
- D4: value LED -> LED Rjo
- R1: renamed from R1 910; value 220 -> 910
- R2: renamed from R2 1K; value 220 -> 1K
Connections:
- A1 pad 11: TRIG 5 -> ECHO 2
- A1 pad 12: TRIG 3 -> TRIG 4
- A1 pad 13: TRIG 2 -> unconnected-(A1-D10-Pad13)
- A1 pad 14: ECHO 1 -> unconnected-(A1-D11-Pad14)
- A1 pad 15: ECHO 2 -> ECHO 4
- A1 pad 19: ECHO 3 -> ECHO 5
- A1 pad 23: ECHO 4 -> SDA
- A1 pad 24: ECHO 5 -> SCL
- J1 pad 1: ECHO 1 -> ECHO 4
- J1 pad 10: TRIG 1 -> TRIG 2
- J1 pad 11: CNY 2 -> ECHO 3
- J1 pad 12: unconnected-(J1-Pin_12-Pad12) -> TRIG 1
- J1 pad 13: CNY 1 -> +5V
- J1 pad 14: unconnected-(J1-Pin_14-Pad14) -> ECHO 1
- J1 pad 15: +5V -> CNY 1
- J1 pad 2: TRIG 2 -> TRIG 4
- J1 pad 3: ECHO 2 -> ECHO 5
- J1 pad 4: TRIG 3 -> SCL
- J1 pad 5: ECHO 3 -> TRIG 5
- J1 pad 6: TRIG 5 -> SDA
- J1 pad 7: ECHO 4 -> CNY 2
- J1 pad 8: TRIG 4 -> ECHO 2
- J1 pad 9: ECHO 5 -> TRIG 3
- U2 pad 16: unconnected-(U2-I15-Pad16) -> TRIG 5
- U2 pad 17: unconnected-(U2-I14-Pad17) -> CNY 2
- U2 pad 18: unconnected-(U2-I13-Pad18) -> TRIG 3
- U2 pad 19: unconnected-(U2-I12-Pad19) -> ECHO 3
- U2 pad 20: CNY 2 -> CNY 1
- U2 pad 21: CNY 1 -> ECHO 1
- U2 pad 23: TRIG 4 -> TRIG 2
Routing:
- net SDA: track 0.00 -> 58.3 mm, vias 0 -> 2
- net SCL: track 0.00 -> 48.4 mm, vias 0 -> 2
- net TRIG 3: track 53.7 -> 25.1 mm
- net TRIG 5: track 55.6 -> 27.6 mm
- net ECHO 3: track 51.2 -> 23.7 mm
- net GND: track 414.4 -> 397.9 mm
- net ECHO 1: track 50.4 -> 35.0 mm
- net ECHO 4: track 41.4 -> 51.4 mm
- net TRIG 4: track 41.4 -> 50.8 mm
- net ECHO 2: track 55.6 -> 61.3 mm
- net TRIG 1: track 35.5 -> 41.1 mm
- net TRIG 2: track 50.4 -> 46.4 mm
- net ECHO 5: track 39.3 -> 43.0 mm
- net +5V: track 267.3 -> 264.0 mm
- net CNY 1: track 23.0 -> 19.9 mm
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Other:
- board text removed: "+"

Commit message: Principal erminada
Parts:
- Dip Switch: renamed from SW2
- renumbered J3 to 24V, SW3 to Arranque, A1 to Nano, J6 to XT60
Routing:
- net ECHO 4: track 51.4 -> 56.5 mm
- net TRIG 4: track 50.8 -> 52.2 mm
Other:
- board text added: "+"
- board text added: "-"
- board text added: "1K"
- board text added: "910"
- board text added: "Led Azul"
- board text added: "Led Rojo"
- board text added: "ON/OFF"
- board text added: "Power Monster"

Commit message: terminava v7
Parts:
- SW2: renamed from Dip Switch
- moved A1 0.57 mm to (170.6, 73.8)
- renumbered Nano to A1, 24V to J3, XT60 to J6, Arranque to SW3
Connections:
- A1 pad 13: unconnected-(A1-D10-Pad13) -> ECHO 4
- A1 pad 14: unconnected-(A1-D11-Pad14) -> ECHO 5
- A1 pad 15: ECHO 4 -> Arranque
- A1 pad 16: Arranque -> Multiplexor Com
- A1 pad 19: ECHO 5 -> Multiplexor S0
- A1 pad 20: Multiplexor Com -> Multiplexor S1
- A1 pad 21: Multiplexor S0 -> Multiplexor S2
- A1 pad 22: Multiplexor S1 -> Multiplexor S3
- A1 pad 25: Multiplexor S2 -> unconnected-(A1-A6-Pad25)
- A1 pad 26: Multiplexor S3 -> unconnected-(A1-A7-Pad26)
Routing:
- net Arranque: track 16.8 -> 35.9 mm
- net ECHO 5: track 43.0 -> 54.2 mm
- net Multiplexor S2: track 10.1 -> 20.6 mm
- net Multiplexor S3: track 6.26 -> 16.2 mm
- net Multiplexor Com: track 27.1 -> 36.8 mm
- net Multiplexor S1: track 8.25 -> 13.0 mm
- net Multiplexor S0: track 12.2 -> 16.7 mm
- net ECHO 4: track 56.5 -> 52.3 mm
- net DIP 5: track 11.1 -> 10.3 mm
- net TRIG 4: track 52.2 -> 52.8 mm
- net SCL: track 48.4 -> 47.8 mm
- net ECHO 2: track 61.3 -> 61.9 mm
- net +5V: track 264.0 -> 264.6 mm
- net SDA: track 58.3 -> 57.7 mm
- net PWM A MONSTER SHIELD: track 5.08 -> 4.57 mm
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Other:
- board size 121 x 65.4 mm -> 121 x 65.9 mm
