File: Electronica/PCB/PCB Principal V7 - V2/PCB Principal V7.kicad_pcb (KiCad board)
At the start: 2 copper layers, 121 x 65.9 mm, 17 parts, among them J1 Conexion Sensores, J2 Power Monster, J3 On/Off General, J6 Power Input 1, SW1 On/Off Motores, SW2 SW_DIP_x05, SW3 SW_Push, U2 CD74HC4067M

Commit message: gnd
Routing:
- net GND: track 398.0 -> 413.5 mm, vias 6 -> 8
Changed lines of the file:
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@@
+	)
+	(gr_line
+		(start 198.4 58.425)
+		(end 198.45 50.575)
+		(stroke
+			(width 0.700001)
+			(type default)
+		)
+		(layer "F.SilkS")
 	)
 	(gr_line
@@
 	)
 	(gr_line
-		(start 198.4 58.375)
-		(end 171.675 58.425)
-		(stroke
-			(width 0.700001)
-			(type default)
-		)
-		(layer "F.SilkS")
-	)
-	(gr_line
 		(start 121.425 88.725)
 		(end 121.425 93.8)
@@
 		(layer "F.SilkS")
 	)
+	(gr_line
+		(start 168.475 55.1)
+		(end 168.5 50.625)
+		(stroke
+			(width 0.700001)
+			(type default)
+		)
+		(layer "F.SilkS")
+	)
 	(gr_rect
 		(start 84.35 46.9)
@@
 	)
 	(segment
+		(start 168.5 55.1)
+		(end 168.5 55.05)
+		(width 0.6)
+		(layer "F.Cu")
+		(net 10)
+	)
+	(segment
+		(start 168.5 50.775)
+		(end 168.525 50.75)
+		(width 0.6)
+		(layer "F.Cu")
+		(net 10)
+	)
+	(segment
 		(start 183.944463 67.8)
 		(end 184.144463 68)
@@
 	)
 	(segment
-		(start 171.775 58.375)
-		(end 171.7 58.45)
+		(start 198.375 58.36)
+		(end 198.39 58.375)
 		(width 0.6)
 		(layer "F.Cu")
@@
 	)
 	(segment
-		(start 198.39 58.375)
-		(end 171.775 58.375)
+		(start 168.5 55.05)
+		(end 168.5 50.775)
+		(width 0.6)
+		(layer "F.Cu")
+		(net 10)
+	)
+	(segment
+		(start 198.375 50.675)
+		(end 198.375 58.36)
 		(width 0.6)
 		(layer "F.Cu")
@@
 	)
 	(via
+		(at 198.375 50.675)
+		(size 1.8)
+		(drill 1)
+		(layers "F.Cu" "B.Cu")
+		(net 10)
+	)
+	(via
 		(at 184.144463 68)
 		(size 1.8)
@@
 	)
 	(via
-		(at 171.7 58.45)
+		(at 168.525 50.75)
+		(size 1.8)
+		(drill 1)
+		(layers "F.Cu" "B.Cu")
+		(net 10)
+	)
+	(via
+		(at 168.5 55.05)
 		(size 1.8)
 		(drill 1)
@@
 	)
 	(segment
-		(start 168.5 58.45)
-		(end 171.7 58.45)
-		(width 1)
-		(layer "B.Cu")
-		(net 10)
-	)
-	(segment
 		(start 150.876 107.694)
 		(end 150.982 107.8)
@@
 	)
 	(segment
+		(start 198.3 50.75)
+		(end 198.375 50.675)
+		(width 0.6)
+		(layer "B.Cu")
+		(net 10)
+	)
+	(segment
 		(start 108.064 67.376)
 		(end 119.436 67.376)
@@
 	)
 	(segment
+		(start 168.5 55.05)
+		(end 168.5 67.9)
+		(width 1)
+		(layer "B.Cu")
+		(net 10)
+	)
+	(segment
 		(start 108.064 107.376)
 		(end 108.064 110.384)
@@
 	)
 	(segment
-		(start 168.5 67.9)
-		(end 168.5 58.45)
-		(width 1)
-		(layer "B.Cu")
-		(net 10)
-	)
-	(segment
 		(start 134.67 102.18)
 		(end 129.54 102.18)
@@
 		(layer "B.Cu")
 		(net 10)
+	)
+	(segment
+		(start 168.525 50.75)
+		(end 198.3 50.75)
+		(width 0.6)
+		(layer "B.Cu")
+		(net 10)

Commit message: Modelos 3D hechos
Parts:
- moved J2 5.09 mm to (124.5, 105.7), turned to 0 degrees
Routing:
- net +5V: track 264.6 -> 262.3 mm
- net GND: track 413.5 -> 412.7 mm

Commit message: ,
Parts:
- added D5: Verde, LED_THT:LED_D5.0mm_Clear, F.Cu at (171.4, 54.7)
- added R3: 120, Resistor_THT:R_Axial_DIN0204_L3.6mm_D1.6mm_P7.62mm_Horizontal, F.Cu at (170.2, 60.2)
Routing:
- net TRIG 2: track 46.4 -> 61.0 mm
- net Net-(D5-K): track 0.00 -> 6.01 mm
