File: Electronica/PCB/PCB Principal V7 - V2/PCB Principal V7.kicad_sch (KiCad schematic)
At the start: 17 parts, among them J1 Conexion Sensores, J2 Power Monster, J3 On/Off General, J6 Power Input 1, SW1 On/Off Motores, SW2 SW_DIP_x05, SW3 SW_Push, U2 CD74HC4067M

Commit message: .
Parts:
- D4: value LED -> LED Rjo
- R1: value 220 -> 910
- R2: value 220 -> 1K
Changed lines of the file:
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@@
 			)
 		)
-		(property "Value" "LED"
+		(property "Value" "LED Rjo"
 			(at 61.214 116.332 0)
 			(effects
@@
 			)
 		)
-		(property "Value" "220"
+		(property "Value" "1K"
 			(at 69.088 118.618 0)
 			(effects
@@
 			)
 		)
-		(property "Value" "220"
+		(property "Value" "910"
 			(at 111.76 100.3299 0)
 			(effects

Commit message: Sensores V3
Parts:
- J1: footprint Connector_PinHeader_2.54mm:PinHeader_2x08_P2.54mm_Horizontal -> Connector_PinHeader_2.54mm:PinHeader_2x08_P2.54mm_Vertical
Connections:
- net +5V: now also J1.13 (Pin_13); no longer J1.15 (Pin_15)
- net CNY 1: now also J1.15 (Pin_15); no longer J1.13 (Pin_13)
- net CNY 2: now also J1.7 (Pin_7); no longer J1.11 (Pin_11)
- net ECHO 1: now also J1.14 (Pin_14); no longer J1.1 (Pin_1)
- net ECHO 2: now also J1.8 (Pin_8); no longer J1.3 (Pin_3)
- net ECHO 3: now also J1.11 (Pin_11); no longer J1.5 (Pin_5)
- net ECHO 4: now also J1.1 (Pin_1); no longer J1.7 (Pin_7)
- net ECHO 5: now also J1.3 (Pin_3); no longer J1.9 (Pin_9)
- net TRIG 1: now also J1.12 (Pin_12); no longer J1.10 (Pin_10)
- net TRIG 2: now also J1.10 (Pin_10); no longer J1.2 (Pin_2)
- net TRIG 3: now also J1.9 (Pin_9); no longer J1.4 (Pin_4)
- net TRIG 4: now also J1.2 (Pin_2); no longer J1.8 (Pin_8)
- net TRIG 5: now also J1.5 (Pin_5); no longer J1.6 (Pin_6)
- new net SCL: J1.4 (Pin_4)
- new net SDA: J1.6 (Pin_6)
- no-connect marks 9 -> 7

Commit message: Placa principal terminada
Parts:
- J1: footprint Connector_PinHeader_2.54mm:PinHeader_2x08_P2.54mm_Vertical -> Connector_PinHeader_2.54mm:PinHeader_2x08_P2.54mm_Horizontal
Connections:
- net CNY 1: now also U2.20 (I11); no longer U2.21 (I10)
- net CNY 2: now also U2.17 (I14); no longer U2.20 (I11)
- net ECHO 1: now also U2.21 (I10); no longer A1.14 (D11)
- net ECHO 2: now also A1.11 (D8); no longer A1.15 (D12)
- net ECHO 3: now also U2.19 (I12); no longer A1.19 (A0)
- net ECHO 4: now also A1.15 (D12); no longer A1.23 (A4)
- net ECHO 5: now also A1.19 (A0); no longer A1.24 (A5)
- net SCL: now also A1.24 (A5)
- net SDA: now also A1.23 (A4)
- net TRIG 2: now also U2.23 (I8); no longer A1.13 (D10)
- net TRIG 3: now also U2.18 (I13); no longer A1.12 (D9)
- net TRIG 4: now also A1.12 (D9); no longer U2.23 (I8)
- net TRIG 5: now also U2.16 (I15); no longer A1.11 (D8)

Commit message: teminada
Connections:
- net Arranque: now also A1.15 (D12); no longer A1.16 (D13)
- net ECHO 4: now also A1.13 (D10); no longer A1.15 (D12)
- net ECHO 5: now also A1.14 (D11); no longer A1.19 (A0)
- net Multiplexor Com: now also A1.16 (D13); no longer A1.20 (A1)
- net Multiplexor S0: now also A1.19 (A0); no longer A1.21 (A2)
- net Multiplexor S1: now also A1.20 (A1); no longer A1.22 (A3)
- net Multiplexor S2: now also A1.21 (A2); no longer A1.25 (A6)
- net Multiplexor S3: now also A1.22 (A3); no longer A1.26 (A7)
- no-connect marks 7 -> 9

Commit message: ,
Parts:
- added D5: Verde, LED_THT:LED_D5.0mm_Clear, symbol Device:LED
- added R3: 120, Resistor_THT:R_Axial_DIN0204_L3.6mm_D1.6mm_P7.62mm_Horizontal, symbol Device:R_US
Connections:
- net GND: now also R3.2
- net TRIG 2: now also D5.2 (A)
- new net: D5.1 (K), R3.1
Other:
- note added: "LED ARRANQUE"
- note removed: "Test Points"
Changed lines of the file:
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@@
 	(wire
 		(pts
+			(xy 41.91 120.65) (xy 44.45 120.65)
+		)
+		(stroke
+			(width 0)
+			(type default)
+		)
+	)
+	(wire
+		(pts
 			(xy 146.05 87.63) (xy 137.16 87.63)
 		)
@@
 		)
 	)
-	(text "Test Points\n"
+	(text "LED ARRANQUE"
 		(exclude_from_sim no)
 		(at 19.304 111.252 0)
@@
 		)
 	)
+	(global_label "TRIG 2"
+		(shape input)
+		(at 26.67 120.65 180)
+		(fields_autoplaced yes)
+		(effects
+			(font
+				(size 1.27 1.27)
+			)
+			(justify right)
+		)
+		(property "Intersheetrefs" "${INTERSHEET_REFS}"
+			(at 17.3953 120.65 0)
+			(effects
+				(font
+					(size 1.27 1.27)
+				)
+				(justify right)
+				(hide yes)
+			)
+		)
+	)
 	(global_label "Multiplexor Com"
 		(shape input)
@@
 	)
 	(symbol
+		(lib_id "power:GND")
+		(at 44.45 120.65 0)
+		(unit 1)
+		(exclude_from_sim no)
+		(in_bom yes)
+		(on_board yes)
+		(dnp no)
+		(fields_autoplaced yes)
+		(property "Reference" "#PWR013"
+			(at 44.45 127 0)
+			(effects
+				(font
+					(size 1.27 1.27)
+				)
+				(hide yes)
+			)
+		)
+		(property "Value" "GND"
+			(at 44.45 125.73 0)
+			(effects
+				(font
+					(size 1.27 1.27)
+				)
+			)
+		)
+		(property "Footprint" ""
+			(at 44.45 120.65 0)
+			(effects
+				(font
+					(size 1.27 1.27)
+				)
+				(hide yes)
+			)
+		)
+		(property "Datasheet" ""
+			(at 44.45 120.65 0)
+			(effects
+				(font
+					(size 1.27 1.27)
+				)
+				(hide yes)
+			)
+		)
+		(property "Description" "Power symbol creates a global label with name \"GND\" , ground"
+			(at 44.45 120.65 0)
+			(effects
+				(font
+					(size 1.27 1.27)
+				)
+				(hide yes)
+			)
+		)
+		(pin "1"
+		)
+		(instances
+			(project "PCB Principal V7"
+				(path "/feeeb2cb-e374-40f4-b9c7-40ed321ecf02"
+					(reference "#PWR013")
+					(unit 1)
+				)
+			)
+		)
+	)
+	(symbol
 		(lib_id "Device:LED")
 		(at 60.96 113.03 0)
@@
 	)
 	(symbol
+		(lib_id "Device:LED")
+		(at 30.48 120.65 180)
+		(unit 1)
+		(exclude_from_sim no)
+		(in_bom yes)
+		(on_board yes)
+		(dnp no)
+		(property "Reference" "D5"
+			(at 30.226 118.364 0)
+			(effects
+				(font
+					(size 1.27 1.27)
+				)
+			)
+		)
+		(property "Value" "Verde"
+			(at 30.226 123.952 0)
+			(effects
+				(font
+					(size 1.27 1.27)
+				)
+			)
+		)
+		(property "Footprint" "LED_THT:LED_D5.0mm_Clear"
+			(at 30.48 120.65 0)
+			(effects
+				(font
+					(size 1.27 1.27)
+				)
+				(hide yes)
+			)
+		)
+		(property "Datasheet" "~"
+			(at 30.48 120.65 0)
+			(effects
+				(font
+					(size 1.27 1.27)
+				)
+				(hide yes)
+			)
+		)
+		(property "Description" "Light emitting diode"
+			(at 30.48 120.65 0)
+			(effects
+				(font
+					(size 1.27 1.27)
+				)
+				(hide yes)
+			)
+		)
+		(pin "1"
+		)
+		(pin "2"
+		)
+		(instances
+			(project "PCB Principal V7"
+				(path "/feeeb2cb-e374-40f4-b9c7-40ed321ecf02"
+					(reference "D5")
+					(unit 1)
+				)
+			)
+		)
+	)
+	(symbol
 		(lib_id "Connector:Screw_Terminal_01x02")
 		(at 54.61 123.19 180)
@@
 					(unit 1)
 				)
+			)
+		)
+	)
+	(symbol
+		(lib_id "Device:R_US")
+		(at 38.1 120.65 90)
+		(mirror x)
+		(unit 1)
+		(exclude_from_sim no)
+		(in_bom yes)
+		(on_board yes)
+		(dnp no)
+		(property "Reference" "R3"
+			(at 38.1 115.57 90)
+			(effects
+				(font
+					(size 1.27 1.27)
+				)
+			)
+		)
+		(property "Value" "120"
+			(at 38.1 118.11 90)
+			(effects
+				(font
+					(size 1.27 1.27)
+				)
+			)
+		)
+		(property "Footprint" "Resistor_THT:R_Axial_DIN0204_L3.6mm_D1.6mm_P7.62mm_Horizontal"
+			(at 38.354 121.666 90)
+			(effects
+				(font
+					(size 1.27 1.27)
+				)
+				(hide yes)
+			)
+		)
+		(property "Datasheet" "~"
+			(at 38.1 120.65 0)
+			(effects
+				(font
+					(size 1.27 1.27)
+				)
+				(hide yes)
+			)
+		)
+		(property "Description" "Resistor, US symbol"
+			(at 38.1 120.65 0)
+			(effects
+				(font
+					(size 1.27 1.27)
+				)
+				(hide yes)
+			)
+		)
+		(pin "1"
+		)
+		(pin "2"
+		)
+		(instances
+			(project "PCB Principal V7"
+				(path "/feeeb2cb-e374-40f4-b9c7-40ed321ecf02"
+					(reference "R3")
+					(unit 1)
+				)
